File: megasequencer/brain/brain/file5E3019D7.sch (KiCad schematic (older format))
At the start: 1 part, among them J1 EURO_PWR_2x5

Commit message: Add pwr, more inputs and outputs
Parts:
- added C5, C6, C7: 10uF, Capacitor_THT:CP_Radial_D5.0mm_P2.00mm, symbol Device:CP
- added R41, R42: R, Resistor_THT:R_Axial_DIN0204_L3.6mm_D1.6mm_P7.62mm_Horizontal, symbol Device:R
- added U4: 78L05, Package_TO_SOT_THT:TO-220-3_Vertical, symbol eurocad:78L05
Connections:
- net +12V: now also C5.1, R41.1, U4.1 (VI_1); no longer J1.1 (+12V), J1.2 (+12V)
- net -12V: now also C6.2, R42.1; no longer J1.10 (-12V), J1.9 (-12V)
- net GND: no longer J1.4 (GND), J1.6 (GND), J1.8 (GND)
- new net: C5.2, C7.2, J1.4 (GND), J1.6 (GND), J1.8 (GND), U4.2 (GND_2)
- new net: J1.1 (+12V), J1.2 (+12V), R41.2
- new net: J1.10 (-12V), J1.9 (-12V), R42.2
- new net +5V: C7.1, U4.3 (VO_3)
Other:
- moved on the sheet: J1
