File: megasequencer/brain/brain/file5E3019D7.sch (KiCad schematic (older format))
At the start: 7 parts, among them J1 EURO_PWR_2x5, U4 78L05

Commit message: Brain seem ok now, also start charting the program
Parts:
- J4: renamed from J1; footprint (none) -> Connector_PinHeader_2.54mm:PinHeader_2x05_P2.54mm_Vertical
- renumbered C5 to C1, C6 to C2, C7 to C3, R41 to R2, R42 to R3, U4 to U1
Changed lines of the file:
@@
 P 2300 4000
 AR Path="/5E353385" Ref="J?"  Part="1"
-AR Path="/5E3019D8/5E353385" Ref="J1"  Part="1"
-F 0 "J1" H 2300 4447 60  0000 C CNN
+AR Path="/5E3019D8/5E353385" Ref="J4"  Part="1"
+F 0 "J4" H 2300 4447 60  0000 C CNN
 F 1 "EURO_PWR_2x5" H 2300 4341 60  0000 C CNN
-F 2 "" H 2300 4000 60  0000 C CNN
+F 2 "Connector_PinHeader_2.54mm:PinHeader_2x05_P2.54mm_Vertical" H 2300 4750 60  0000 C CNN
 F 3 "" H 2300 4000 60  0000 C CNN
 	1    2300 4000
@@
 P 1650 4000
 AR Path="/5E353392" Ref="#PWR?"  Part="1"
-AR Path="/5E3019D8/5E353392" Ref="#PWR02"  Part="1"
-F 0 "#PWR02" H 1650 3750 50  0001 C CNN
+AR Path="/5E3019D8/5E353392" Ref="#PWR08"  Part="1"
+F 0 "#PWR08" H 1650 3750 50  0001 C CNN
 F 1 "GND" V 1655 3872 50  0000 R CNN
 F 2 "" H 1650 4000 50  0001 C CNN
@@
 P 5200 3200
 AR Path="/5DDE016B" Ref="#PWR?"  Part="1"
-AR Path="/5E3019D8/5DDE016B" Ref="#PWR01"  Part="1"
-F 0 "#PWR01" H 5200 3050 50  0001 C CNN
+AR Path="/5E3019D8/5DDE016B" Ref="#PWR09"  Part="1"
+F 0 "#PWR09" H 5200 3050 50  0001 C CNN
 F 1 "+12V" V 5215 3328 50  0000 L CNN
 F 2 "" H 5200 3200 50  0001 C CNN
@@
 P 5200 4800
 AR Path="/5DDE017E" Ref="#PWR?"  Part="1"
-AR Path="/5E3019D8/5DDE017E" Ref="#PWR03"  Part="1"
-F 0 "#PWR03" H 5200 4900 50  0001 C CNN
+AR Path="/5E3019D8/5DDE017E" Ref="#PWR010"  Part="1"
+F 0 "#PWR010" H 5200 4900 50  0001 C CNN
 F 1 "-12V" V 5215 4928 50  0000 L CNN
 F 2 "" H 5200 4800 50  0001 C CNN
@@
 $EndComp
 $Comp
-L Device:CP C5
+L Device:CP C1
 U 1 1 5DDE01E5
 P 4700 3750
-F 0 "C5" H 4818 3796 50  0000 L CNN
+F 0 "C1" H 4818 3796 50  0000 L CNN
 F 1 "10uF" H 4818 3705 50  0000 L CNN
 F 2 "Capacitor_THT:CP_Radial_D5.0mm_P2.00mm" H 4738 3600 50  0001 C CNN
@@
 $EndComp
 $Comp
-L Device:CP C6
+L Device:CP C2
 U 1 1 5DDE02B9
 P 4700 4250
-F 0 "C6" H 4818 4296 50  0000 L CNN
+F 0 "C2" H 4818 4296 50  0000 L CNN
 F 1 "10uF" H 4818 4205 50  0000 L CNN
 F 2 "Capacitor_THT:CP_Radial_D5.0mm_P2.00mm" H 4738 4100 50  0001 C CNN
@@
 $EndComp
 $Comp
-L Device:R R41
+L Device:R R2
 U 1 1 5DDE0A8B
 P 4350 3500
-F 0 "R41" V 4143 3500 50  0000 C CNN
+F 0 "R2" V 4143 3500 50  0000 C CNN
 F 1 "R" V 4234 3500 50  0000 C CNN
 F 2 "Resistor_THT:R_Axial_DIN0204_L3.6mm_D1.6mm_P7.62mm_Horizontal" V 4280 3500 50  0001 C CNN
@@
 $EndComp
 $Comp
-L Device:R R42
+L Device:R R3
 U 1 1 5DDE0B7D
 P 4350 4500
-F 0 "R42" V 4143 4500 50  0000 C CNN
+F 0 "R3" V 4143 4500 50  0000 C CNN
 F 1 "R" V 4234 4500 50  0000 C CNN
 F 2 "Resistor_THT:R_Axial_DIN0204_L3.6mm_D1.6mm_P7.62mm_Horizontal" V 4280 4500 50  0001 C CNN
@@
 $EndComp
 $Comp
-L brain-rescue:78L05-eurocad U4
+L brain-rescue:78L05-eurocad U1
 U 1 1 5DDE108A
 P 6150 3550
-F 0 "U4" H 6150 4047 50  0000 C CNN
+F 0 "U1" H 6150 4047 50  0000 C CNN
 F 1 "78L05" H 6150 3956 50  0000 C CNN
 F 2 "Package_TO_SOT_THT:TO-220-3_Vertical" H 6150 3865 50  0000 C CNN
@@
 Connection ~ 4700 4000
 $Comp
-L Device:CP C7
+L Device:CP C3
 U 1 1 5DDE4E43
 P 6800 3750
-F 0 "C7" H 6918 3796 50  0000 L CNN
+F 0 "C3" H 6918 3796 50  0000 L CNN
 F 1 "10uF" H 6918 3705 50  0000 L CNN
 F 2 "Capacitor_THT:CP_Radial_D5.0mm_P2.00mm" H 6838 3600 50  0001 C CNN
@@
 $EndComp
 $Comp
-L power:+5V #PWR04
+L power:+5V #PWR011
 U 1 1 5DDE4EC7
 P 7050 3500
-F 0 "#PWR04" H 7050 3350 50  0001 C CNN
+F 0 "#PWR011" H 7050 3350 50  0001 C CNN
 F 1 "+5V" V 7065 3628 50  0000 L CNN
 F 2 "" H 7050 3500 50  0001 C CNN

Commit message: Almost done now with both pcbs
Parts:
- R2, R3: value R -> 10
- U1: footprint Package_TO_SOT_THT:TO-220-3_Vertical -> Package_TO_SOT_THT:TO-220-3_Horizontal_TabDown
Connections:
- net GND: now also C1.2, C2.1, C3.2, J4.4 (GND), J4.6 (GND), J4.8 (GND), U1.2 (GND_2)
Changed lines of the file:
@@
 	1    0    0    -1
-$EndComp
-$Comp
-L power:GND #PWR?
-U 1 1 5E353392
-P 1650 4000
-AR Path="/5E353392" Ref="#PWR?"  Part="1"
-AR Path="/5E3019D8/5E353392" Ref="#PWR08"  Part="1"
-F 0 "#PWR08" H 1650 3750 50  0001 C CNN
-F 1 "GND" V 1655 3872 50  0000 R CNN
-F 2 "" H 1650 4000 50  0001 C CNN
-F 3 "" H 1650 4000 50  0001 C CNN
-	1    1650 4000
-	0    1    1    0
 $EndComp
 Wire Wire Line
@@
 P 4350 3500
 F 0 "R2" V 4143 3500 50  0000 C CNN
-F 1 "R" V 4234 3500 50  0000 C CNN
+F 1 "10" V 4234 3500 50  0000 C CNN
 F 2 "Resistor_THT:R_Axial_DIN0204_L3.6mm_D1.6mm_P7.62mm_Horizontal" V 4280 3500 50  0001 C CNN
 F 3 "~" H 4350 3500 50  0001 C CNN
@@
 P 4350 4500
 F 0 "R3" V 4143 4500 50  0000 C CNN
-F 1 "R" V 4234 4500 50  0000 C CNN
+F 1 "10" V 4234 4500 50  0000 C CNN
 F 2 "Resistor_THT:R_Axial_DIN0204_L3.6mm_D1.6mm_P7.62mm_Horizontal" V 4280 4500 50  0001 C CNN
 F 3 "~" H 4350 4500 50  0001 C CNN
@@
 F 0 "U1" H 6150 4047 50  0000 C CNN
 F 1 "78L05" H 6150 3956 50  0000 C CNN
-F 2 "Package_TO_SOT_THT:TO-220-3_Vertical" H 6150 3865 50  0000 C CNN
+F 2 "Package_TO_SOT_THT:TO-220-3_Horizontal_TabDown" H 6150 3865 50  0000 C CNN
 F 3 "regulator\\lm78lxx.pdf" H 6150 3774 50  0000 C CNN
 	1    6150 3550
@@
 Wire Wire Line
 	4700 4000 4700 4100
+$Comp
+L power:GND #PWR?
+U 1 1 5E353392
+P 1650 4000
+AR Path="/5E353392" Ref="#PWR?"  Part="1"
+AR Path="/5E3019D8/5E353392" Ref="#PWR08"  Part="1"
+F 0 "#PWR08" H 1650 3750 50  0001 C CNN
+F 1 "GND" V 1655 3872 50  0000 R CNN
+F 2 "" H 1650 4000 50  0001 C CNN
+F 3 "" H 1650 4000 50  0001 C CNN
+	1    1650 4000
+	0    1    1    0
+$EndComp
+$Comp
+L power:GND #PWR?
+U 1 1 5E36115A
+P 6150 4175
+AR Path="/5E36115A" Ref="#PWR?"  Part="1"
+AR Path="/5E3019D8/5E36115A" Ref="#PWR0103"  Part="1"
+F 0 "#PWR0103" H 6150 3925 50  0001 C CNN
+F 1 "GND" H 6225 4000 50  0000 R CNN
+F 2 "" H 6150 4175 50  0001 C CNN
+F 3 "" H 6150 4175 50  0001 C CNN
+	1    6150 4175
+	1    0    0    -1
+$EndComp
+Wire Wire Line
+	6150 4000 6150 4175
 $EndSCHEMATC
