File: megasequencer/brain/brain/file5E366866.sch (KiCad schematic (older format))
At the start: 1 part, among them U1 ATmega328P-PU

Commit message: Add pwr, more inputs and outputs
Connections:
- net labels added: PULSE_LENGTH_5V
Changed lines of the file:
@@
 $Descr A4 11693 8268
 encoding utf-8
-Sheet 4 6
+Sheet 4 7
 Title ""
 Date ""
@@
 Text HLabel 4450 2350 2    50   Input ~ 0
 SEQ_ZERO
+Text HLabel 4500 3350 2    50   Input ~ 0
+PULSE_LENGTH_5V
 $EndSCHEMATC
