File: megasequencer/brain/brain/file5E366866.sch (KiCad schematic (older format))
At the start: 1 part, among them U1 ATmega328P-PU

Commit message: Finish interface and continue with brain
Parts:
- added J3: ICSP, Connector_PinHeader_2.54mm:PinHeader_2x05_P2.54mm_Vertical, symbol Connector_Generic:Conn_02x05_Odd_Even
Connections:
- wire segments 27 -> 36
- no-connect marks 0 -> 1
Changed lines of the file:
@@
 $Descr A4 11693 8268
 encoding utf-8
-Sheet 4 7
+Sheet 3 6
 Title ""
 Date ""
@@
 Text HLabel 4500 4250 2    50   Output ~ 0
 STEPS_LATCH
+$Comp
+L Connector_Generic:Conn_02x05_Odd_Even J3
+U 1 1 5E08B37C
+P 7725 2275
+F 0 "J3" H 7775 2692 50  0000 C CNN
+F 1 "ICSP" H 7775 2601 50  0000 C CNN
+F 2 "Connector_PinHeader_2.54mm:PinHeader_2x05_P2.54mm_Vertical" H 7725 2275 50  0001 C CNN
+F 3 "~" H 7725 2275 50  0001 C CNN
+	1    7725 2275
+	1    0    0    -1
+$EndComp
+Text Label 7525 2475 2    50   ~ 0
+D12-MISO
+Text Label 7525 2375 2    50   ~ 0
+D13-SCK
+Text Label 7525 2275 2    50   ~ 0
+RST
+Text Label 7525 2075 2    50   ~ 0
+D11-MOSI
+$Comp
+L power:+5V #PWR?
+U 1 1 5E08BEE4
+P 8250 2075
+AR Path="/5E08BEE4" Ref="#PWR?"  Part="1"
+AR Path="/5E366867/5E08BEE4" Ref="#PWR08"  Part="1"
+F 0 "#PWR08" H 8250 1925 50  0001 C CNN
+F 1 "+5V" H 8400 2125 50  0000 C CNN
+F 2 "" H 8250 2075 50  0001 C CNN
+F 3 "" H 8250 2075 50  0001 C CNN
+	1    8250 2075
+	0    1    1    0
+$EndComp
+Wire Wire Line
+	8025 2075 8250 2075
+$Comp
+L power:GND #PWR?
+U 1 1 5E08CAE8
+P 8175 2550
+AR Path="/5E08CAE8" Ref="#PWR?"  Part="1"
+AR Path="/5E366867/5E08CAE8" Ref="#PWR07"  Part="1"
+F 0 "#PWR07" H 8175 2300 50  0001 C CNN
+F 1 "GND" H 8180 2377 50  0000 C CNN
+F 2 "" H 8175 2550 50  0001 C CNN
+F 3 "" H 8175 2550 50  0001 C CNN
+	1    8175 2550
+	1    0    0    -1
+$EndComp
+Wire Wire Line
+	8025 2175 8175 2175
+Wire Wire Line
+	8175 2175 8175 2275
+Wire Wire Line
+	8025 2275 8175 2275
+Connection ~ 8175 2275
+Wire Wire Line
+	8175 2275 8175 2375
+Wire Wire Line
+	8025 2375 8175 2375
+Connection ~ 8175 2375
+Wire Wire Line
+	8175 2375 8175 2475
+Connection ~ 8175 2475
+Wire Wire Line
+	8175 2475 8175 2550
+Wire Wire Line
+	8025 2475 8175 2475
+NoConn ~ 7525 2175
 $EndSCHEMATC

Commit message: Brain seem ok now, also start charting the program
Parts:
- renumbered J3 to J5, U1 to U2
Changed lines of the file:
@@
 P 2850 3350
 AR Path="/5E36C56A" Ref="U?"  Part="1"
-AR Path="/5E366867/5E36C56A" Ref="U1"  Part="1"
-F 0 "U1" H 2209 3396 50  0000 R CNN
+AR Path="/5E366867/5E36C56A" Ref="U2"  Part="1"
+F 0 "U2" H 2209 3396 50  0000 R CNN
 F 1 "ATmega328P-PU" H 2209 3305 50  0000 R CNN
 F 2 "Package_DIP:DIP-28_W7.62mm" H 2850 3350 50  0001 C CIN
@@
 P 2150 2150
 AR Path="/5E36C583" Ref="#PWR?"  Part="1"
-AR Path="/5E366867/5E36C583" Ref="#PWR09"  Part="1"
-F 0 "#PWR09" H 2150 2000 50  0001 C CNN
+AR Path="/5E366867/5E36C583" Ref="#PWR012"  Part="1"
+F 0 "#PWR012" H 2150 2000 50  0001 C CNN
 F 1 "+5V" V 2165 2278 50  0000 L CNN
 F 2 "" H 2150 2150 50  0001 C CNN
@@
 P 2850 1750
 AR Path="/5E36C589" Ref="#PWR?"  Part="1"
-AR Path="/5E366867/5E36C589" Ref="#PWR010"  Part="1"
-F 0 "#PWR010" H 2850 1600 50  0001 C CNN
+AR Path="/5E366867/5E36C589" Ref="#PWR013"  Part="1"
+F 0 "#PWR013" H 2850 1600 50  0001 C CNN
 F 1 "+5V" H 2700 1800 50  0000 C CNN
 F 2 "" H 2850 1750 50  0001 C CNN
@@
 P 2950 1750
 AR Path="/5E36C58F" Ref="#PWR?"  Part="1"
-AR Path="/5E366867/5E36C58F" Ref="#PWR012"  Part="1"
-F 0 "#PWR012" H 2950 1600 50  0001 C CNN
+AR Path="/5E366867/5E36C58F" Ref="#PWR015"  Part="1"
+F 0 "#PWR015" H 2950 1600 50  0001 C CNN
 F 1 "+5V" H 3100 1800 50  0000 C CNN
 F 2 "" H 2950 1750 50  0001 C CNN
@@
 P 2850 4950
 AR Path="/5E36C598" Ref="#PWR?"  Part="1"
-AR Path="/5E366867/5E36C598" Ref="#PWR011"  Part="1"
-F 0 "#PWR011" H 2850 4700 50  0001 C CNN
+AR Path="/5E366867/5E36C598" Ref="#PWR014"  Part="1"
+F 0 "#PWR014" H 2850 4700 50  0001 C CNN
 F 1 "GND" H 2855 4777 50  0000 C CNN
 F 2 "" H 2850 4950 50  0001 C CNN
@@
 STEPS_LATCH
 $Comp
-L Connector_Generic:Conn_02x05_Odd_Even J3
+L Connector_Generic:Conn_02x05_Odd_Even J5
 U 1 1 5E08B37C
 P 7725 2275
-F 0 "J3" H 7775 2692 50  0000 C CNN
+F 0 "J5" H 7775 2692 50  0000 C CNN
 F 1 "ICSP" H 7775 2601 50  0000 C CNN
 F 2 "Connector_PinHeader_2.54mm:PinHeader_2x05_P2.54mm_Vertical" H 7725 2275 50  0001 C CNN
@@
 P 8250 2075
 AR Path="/5E08BEE4" Ref="#PWR?"  Part="1"
-AR Path="/5E366867/5E08BEE4" Ref="#PWR08"  Part="1"
-F 0 "#PWR08" H 8250 1925 50  0001 C CNN
+AR Path="/5E366867/5E08BEE4" Ref="#PWR017"  Part="1"
+F 0 "#PWR017" H 8250 1925 50  0001 C CNN
 F 1 "+5V" H 8400 2125 50  0000 C CNN
 F 2 "" H 8250 2075 50  0001 C CNN
@@
 P 8175 2550
 AR Path="/5E08CAE8" Ref="#PWR?"  Part="1"
-AR Path="/5E366867/5E08CAE8" Ref="#PWR07"  Part="1"
-F 0 "#PWR07" H 8175 2300 50  0001 C CNN
+AR Path="/5E366867/5E08CAE8" Ref="#PWR016"  Part="1"
+F 0 "#PWR016" H 8175 2300 50  0001 C CNN
 F 1 "GND" H 8180 2377 50  0000 C CNN
 F 2 "" H 8175 2550 50  0001 C CNN

Commit message: Almost done now with both pcbs
Parts:
- added C14, C15: 22pF, Capacitor_THT:C_Disc_D3.0mm_W1.6mm_P2.50mm, symbol Device:C
- added C16: 15pF, Capacitor_THT:C_Disc_D3.0mm_W1.6mm_P2.50mm, symbol Device:C
- added C17, C18: 100nF, Capacitor_THT:C_Disc_D3.0mm_W1.6mm_P2.50mm, symbol Device:C
- added D7: 1N4148, Diode_THT:D_A-405_P7.62mm_Horizontal, symbol Device:D
- added FB1, FB2: Ferrite_Bead, Inductor_THT:L_Axial_L6.6mm_D2.7mm_P10.16mm_Horizontal_Vishay_IM-2, symbol Device:Ferrite_Bead
- added R40: 330, Resistor_THT:R_Axial_DIN0207_L6.3mm_D2.5mm_P7.62mm_Horizontal, symbol Device:R
- added R41: 10K, Resistor_THT:R_Axial_DIN0207_L6.3mm_D2.5mm_P7.62mm_Horizontal, symbol Device:R
- added SW1: RST, Button_Switch_THT:SW_PUSH_6mm, symbol Switch:SW_Push
- added Y1: Crystal, Crystal:Crystal_HC18-U_Vertical, symbol Device:Crystal
Connections:
- wire segments 36 -> 57

Commit message: Wrong LED direction
Parts:
- U2: symbol MCU_Microchip_ATmega:ATmega328P-PU -> brain-rescue:ATmega328P-PU-MCU_Microchip_ATmega
Changed lines of the file:
@@
 EESchema Schematic File Version 4
-LIBS:brain-cache
 EELAYER 30 0
 EELAYER END
 $Descr A4 11693 8268
 encoding utf-8
-Sheet 3 5
+Sheet 2 5
 Title ""
 Date ""
@@
 $EndDescr
 $Comp
-L MCU_Microchip_ATmega:ATmega328P-PU U?
+L brain-rescue:ATmega328P-PU-MCU_Microchip_ATmega U?
 U 1 1 5E36C56A
 P 2850 3350
