File: megasequencer/brain/brain/file5E36D63D.sch (KiCad schematic (older format))
At the start: 39 parts, among them J5 EXT_RATE_CV, J8 EXT_POS_CV, J9 PULSE_LENGTH_CV, U2 TL074, U3 TL074

Commit message: Finish interface and continue with brain
Parts:
- removed J5: EXT_RATE_CV, Connector_Audio:Jack_3.5mm_QingPu_WQP-PJ398SM_Vertical_CircularHoles, symbol Connector:AudioJack2_SwitchT
- removed J8: EXT_POS_CV, Connector_Audio:Jack_3.5mm_QingPu_WQP-PJ398SM_Vertical_CircularHoles, symbol Connector:AudioJack2_SwitchT
- removed J9: PULSE_LENGTH_CV, Connector_Audio:Jack_3.5mm_QingPu_WQP-PJ398SM_Vertical_CircularHoles, symbol Connector:AudioJack2_SwitchT
- removed R30, R31, R32, R33, R38, R39: 100K, Resistor_THT:R_Axial_DIN0207_L6.3mm_D2.5mm_P7.62mm_Horizontal, symbol Device:R
- removed RV1: RATE_IN_OFFSET, Potentiometer_THT:Potentiometer_Alps_RK09L_Single_Vertical, symbol Device:R_POT
- removed RV2: EXT_POS_IN_OFFSET, Potentiometer_THT:Potentiometer_Alps_RK09L_Single_Vertical, symbol Device:R_POT
- removed RV3: RATE_IN_ATT, Potentiometer_THT:Potentiometer_Alps_RK09L_Single_Vertical, symbol Device:R_POT
- removed RV4: EXT_POS_IN_ATT, Potentiometer_THT:Potentiometer_Alps_RK09L_Single_Vertical, symbol Device:R_POT
- removed RV5: PULSE_LENGTH_IN_OFFSET, Potentiometer_THT:Potentiometer_Alps_RK09L_Single_Vertical, symbol Device:R_POT
- removed RV6: PULSE_LENGTH_IN_ATT, Potentiometer_THT:Potentiometer_Alps_RK09L_Single_Vertical, symbol Device:R_POT
- U3: value TL074 -> TL072
Connections:
- net labels added: POS_RAW, PULSE_LENGTH_RAW, RATE_RAW
- wire segments 129 -> 87
- no-connect marks 3 -> 0

Commit message: Brain seem ok now, also start charting the program
Parts:
- D1, D2: value D_Schottky -> S
- D3: renamed from D6; value D_Schottky -> S
- D4: renamed from D7; value D_Schottky -> S
- D5: renamed from D11; value D_Schottky -> S
- D6: renamed from D12; value D_Schottky -> S
- renumbered C1 to C4, C2 to C5, C3 to C6, C4 to C7, R24 to R10, R25 to R11, R36 to R12, R26 to R13, R27 to R14, R37 to R15, R20 to R4, R21 to R5, R34 to R6, R22 to R7, R23 to R8, R35 to R9, U2 to U3, U3 to U4

Commit message: Almost done now with both pcbs
Connections:
- net GND: now also U3.10 (+), U3.12 (+); no longer U3.10 (+), U3.12 (+)
- net POS_RAW: now also U3.13 (-); no longer U3.9 (-)
- net at R10.2, R14.1: now also U3.14; no longer U3.8
- net at R10.1, R8.2: now also U3.9 (-); no longer U3.13 (-)
- net at R5.2, R8.1: now also U3.8; no longer U3.14
Changed lines of the file:
@@
 $Comp
 L Amplifier_Operational:TL074 U?
-U 3 1 5E36F06C
+U 4 1 5E36F06C
 P 3900 4100
 AR Path="/5E36F06C" Ref="U?"  Part="3"
-AR Path="/5E36D63E/5E36F06C" Ref="U3"  Part="3"
+AR Path="/5E36D63E/5E36F06C" Ref="U3"  Part="4"
 F 0 "U3" H 3950 4250 50  0000 C CNN
 F 1 "TL074" H 3950 4350 50  0000 C CNN
 F 2 "Package_DIP:DIP-14_W7.62mm" H 3850 4200 50  0001 C CNN
 F 3 "http://www.ti.com/lit/ds/symlink/tl071.pdf" H 3950 4300 50  0001 C CNN
-	3    3900 4100
+	4    3900 4100
 	-1   0    0    1
 $EndComp
@@
 $Comp
 L Amplifier_Operational:TL074 U?
-U 4 1 5E36F095
+U 3 1 5E36F095
 P 2700 4200
 AR Path="/5E36F095" Ref="U?"  Part="4"
-AR Path="/5E36D63E/5E36F095" Ref="U3"  Part="4"
+AR Path="/5E36D63E/5E36F095" Ref="U3"  Part="3"
 F 0 "U3" H 2750 4350 50  0000 C CNN
 F 1 "TL074" H 2750 4450 50  0000 C CNN
 F 2 "Package_DIP:DIP-14_W7.62mm" H 2650 4300 50  0001 C CNN
 F 3 "http://www.ti.com/lit/ds/symlink/tl071.pdf" H 2750 4400 50  0001 C CNN
-	4    2700 4200
+	3    2700 4200
 	-1   0    0    1
 $EndComp
