File: megasequencer/brain/brain/file5DDEBCF3.sch (KiCad schematic (older format))
At the start: 4 parts, among them U5 74HC595, U6 74HC595

Commit message: Finish interface and continue with brain
Parts:
- added J4: TO_OUTPUTS, Connector_PinHeader_2.54mm:PinHeader_1x17_P2.54mm_Vertical, symbol Connector:Conn_01x17_Male
Connections:
- net GND: now also J4.1 (Pin_1)
- net OUT1: no longer names the net of U5.15 (QA)
- net OUT1: now also J4.2 (Pin_2)
- net OUT10: no longer names the net of U6.1 (QB)
- net OUT10: now also J4.11 (Pin_11)
- net OUT11: no longer names the net of U6.2 (QC)
- net OUT11: now also J4.12 (Pin_12)
- net OUT12: no longer names the net of U6.3 (QD)
- net OUT12: now also J4.13 (Pin_13)
- net OUT13: no longer names the net of U6.4 (QE)
- net OUT13: now also J4.14 (Pin_14)
- net OUT14: no longer names the net of U6.5 (QF)
- net OUT14: now also J4.15 (Pin_15)
- net OUT15: no longer names the net of U6.6 (QG)
- net OUT15: now also J4.16 (Pin_16)
- net OUT16: no longer names the net of U6.7 (QH)
- net OUT16: now also J4.17 (Pin_17)
- net OUT2: no longer names the net of U5.1 (QB)
- net OUT2: now also J4.3 (Pin_3)
- net OUT3: no longer names the net of U5.2 (QC)
- net OUT3: now also J4.4 (Pin_4)
- net OUT4: no longer names the net of U5.3 (QD)
- net OUT4: now also J4.5 (Pin_5)
- net OUT5: no longer names the net of U5.4 (QE)
- net OUT5: now also J4.6 (Pin_6)
- net OUT6: no longer names the net of U5.5 (QF)
- net OUT6: now also J4.7 (Pin_7)
- net OUT7: no longer names the net of U5.6 (QG)
- net OUT7: now also J4.8 (Pin_8)
- net OUT8: no longer names the net of U5.7 (QH)
- net OUT8: now also J4.9 (Pin_9)
- net OUT9: no longer names the net of U6.15 (QA)
- net OUT9: now also J4.10 (Pin_10)
Changed lines of the file:
@@
 $Descr A4 11693 8268
 encoding utf-8
-Sheet 7 7
+Sheet 6 6
 Title ""
 Date ""
@@
 Text Notes 7050 7100 0    50   ~ 0
 https://www.arduino.cc/en/Tutorial/ShiftOut
-Text HLabel 3150 2600 2    50   Output ~ 0
-OUT1
-Text HLabel 3150 2700 2    50   Output ~ 0
-OUT2
-Text HLabel 3150 2800 2    50   Output ~ 0
-OUT3
-Text HLabel 3150 2900 2    50   Output ~ 0
-OUT4
-Text HLabel 3150 3000 2    50   Output ~ 0
-OUT5
-Text HLabel 3150 3100 2    50   Output ~ 0
-OUT6
-Text HLabel 3150 3200 2    50   Output ~ 0
-OUT7
-Text HLabel 3150 3300 2    50   Output ~ 0
-OUT8
-Text HLabel 3150 4650 2    50   Output ~ 0
-OUT9
-Text HLabel 3150 4750 2    50   Output ~ 0
-OUT10
-Text HLabel 3150 4850 2    50   Output ~ 0
-OUT11
-Text HLabel 3150 4950 2    50   Output ~ 0
-OUT12
-Text HLabel 3150 5050 2    50   Output ~ 0
-OUT13
-Text HLabel 3150 5150 2    50   Output ~ 0
-OUT14
-Text HLabel 3150 5250 2    50   Output ~ 0
-OUT15
-Text HLabel 3150 5350 2    50   Output ~ 0
-OUT16
-Wire Wire Line
-	2700 2600 3150 2600
-Wire Wire Line
-	2700 2700 3150 2700
-Wire Wire Line
-	2700 2800 3150 2800
-Wire Wire Line
-	2700 2900 3150 2900
-Wire Wire Line
-	2700 3000 3150 3000
-Wire Wire Line
-	2700 3100 3150 3100
-Wire Wire Line
-	2700 3200 3150 3200
-Wire Wire Line
-	2700 3300 3150 3300
-Wire Wire Line
-	2700 4650 3150 4650
-Wire Wire Line
-	2700 4750 3150 4750
-Wire Wire Line
-	2700 4850 3150 4850
-Wire Wire Line
-	2700 4950 3150 4950
-Wire Wire Line
-	2700 5050 3150 5050
-Wire Wire Line
-	2700 5150 3150 5150
-Wire Wire Line
-	2700 5250 3150 5250
-Wire Wire Line
-	2700 5350 3150 5350
+$Comp
+L Connector:Conn_01x17_Male J?
+U 1 1 5E0643C1
+P 5150 3300
+AR Path="/5E0643C1" Ref="J?"  Part="1"
+AR Path="/5DDEBCF4/5E0643C1" Ref="J4"  Part="1"
+F 0 "J4" H 5122 3324 50  0000 R CNN
+F 1 "TO_OUTPUTS" H 5122 3233 50  0000 R CNN
+F 2 "Connector_PinHeader_2.54mm:PinHeader_1x17_P2.54mm_Vertical" H 5150 3300 50  0001 C CNN
+F 3 "~" H 5150 3300 50  0001 C CNN
+	1    5150 3300
+	-1   0    0    -1
+$EndComp
+Wire Wire Line
+	2700 2600 4950 2600
+Wire Wire Line
+	2700 2700 4950 2700
+Wire Wire Line
+	2700 2800 4950 2800
+Wire Wire Line
+	2700 2900 4950 2900
+Wire Wire Line
+	2700 3000 4950 3000
+Wire Wire Line
+	2700 3100 4950 3100
+Wire Wire Line
+	2700 3200 4950 3200
+Wire Wire Line
+	2700 3300 4950 3300
+Wire Wire Line
+	4000 4650 4000 3400
+Wire Wire Line
+	4000 3400 4950 3400
+Wire Wire Line
+	2700 4650 4000 4650
+Wire Wire Line
+	4100 4750 4100 3500
+Wire Wire Line
+	4100 3500 4950 3500
+Wire Wire Line
+	2700 4750 4100 4750
+Wire Wire Line
+	4200 4850 4200 3600
+Wire Wire Line
+	4200 3600 4950 3600
+Wire Wire Line
+	2700 4850 4200 4850
+Wire Wire Line
+	2700 4950 4300 4950
+Wire Wire Line
+	4300 3700 4950 3700
+Wire Wire Line
+	4300 4950 4300 3700
+Wire Wire Line
+	4400 5050 4400 3800
+Wire Wire Line
+	4400 3800 4950 3800
+Wire Wire Line
+	2700 5050 4400 5050
+Wire Wire Line
+	4500 5150 4500 3900
+Wire Wire Line
+	4500 3900 4950 3900
+Wire Wire Line
+	2700 5150 4500 5150
+Wire Wire Line
+	4600 5250 4600 4000
+Wire Wire Line
+	4600 4000 4950 4000
+Wire Wire Line
+	2700 5250 4600 5250
+Wire Wire Line
+	4700 5350 4700 4100
+Wire Wire Line
+	4700 4100 4950 4100
+Wire Wire Line
+	2700 5350 4700 5350
+$Comp
+L power:GND #PWR016
+U 1 1 5E07C333
+P 4750 2500
+F 0 "#PWR016" H 4750 2250 50  0001 C CNN
+F 1 "GND" V 4755 2372 50  0000 R CNN
+F 2 "" H 4750 2500 50  0001 C CNN
+F 3 "" H 4750 2500 50  0001 C CNN
+	1    4750 2500
+	0    1    1    0
+$EndComp
+Wire Wire Line
+	4750 2500 4950 2500
 $EndSCHEMATC

Commit message: Brain seem ok now, also start charting the program
Parts:
- renumbered J4 to J6
Changed lines of the file:
@@
 $Descr A4 11693 8268
 encoding utf-8
-Sheet 6 6
+Sheet 5 6
 Title ""
 Date ""
@@
 $EndDescr
 $Comp
-L power:+5V #PWR0101
+L power:+5V #PWR040
 U 1 1 5DDEC4E8
 P 2300 2150
-F 0 "#PWR0101" H 2300 2000 50  0001 C CNN
+F 0 "#PWR040" H 2300 2000 50  0001 C CNN
 F 1 "+5V" H 2315 2323 50  0000 C CNN
 F 2 "" H 2300 2150 50  0001 C CNN
@@
 	2300 2150 2300 2400
 $Comp
-L power:+5V #PWR0102
+L power:+5V #PWR042
 U 1 1 5DDEC7AF
 P 2300 4200
-F 0 "#PWR0102" H 2300 4050 50  0001 C CNN
+F 0 "#PWR042" H 2300 4050 50  0001 C CNN
 F 1 "+5V" H 2315 4373 50  0000 C CNN
 F 2 "" H 2300 4200 50  0001 C CNN
@@
 	2300 4200 2300 4300
 $Comp
-L power:GND #PWR0103
+L power:GND #PWR041
 U 1 1 5DDEC816
 P 2300 3750
-F 0 "#PWR0103" H 2300 3500 50  0001 C CNN
+F 0 "#PWR041" H 2300 3500 50  0001 C CNN
 F 1 "GND" H 2305 3577 50  0000 C CNN
 F 2 "" H 2300 3750 50  0001 C CNN
@@
 $EndComp
 $Comp
-L power:GND #PWR0104
+L power:GND #PWR043
 U 1 1 5DDEC82E
 P 2300 5800
-F 0 "#PWR0104" H 2300 5550 50  0001 C CNN
+F 0 "#PWR043" H 2300 5550 50  0001 C CNN
 F 1 "GND" H 2305 5627 50  0000 C CNN
 F 2 "" H 2300 5800 50  0001 C CNN
@@
 Connection ~ 2600 4300
 $Comp
-L power:+5V #PWR0105
+L power:+5V #PWR036
 U 1 1 5DDEDEA1
 P 1750 2900
-F 0 "#PWR0105" H 1750 2750 50  0001 C CNN
+F 0 "#PWR036" H 1750 2750 50  0001 C CNN
 F 1 "+5V" V 1765 3028 50  0000 L CNN
 F 2 "" H 1750 2900 50  0001 C CNN
@@
 $EndComp
 $Comp
-L power:+5V #PWR0106
+L power:+5V #PWR038
 U 1 1 5DDEDEC0
 P 1750 4950
-F 0 "#PWR0106" H 1750 4800 50  0001 C CNN
+F 0 "#PWR038" H 1750 4800 50  0001 C CNN
 F 1 "+5V" V 1765 5078 50  0000 L CNN
 F 2 "" H 1750 4950 50  0001 C CNN
@@
 	1750 4950 1900 4950
 $Comp
-L power:GND #PWR0107
+L power:GND #PWR037
 U 1 1 5DDEE044
 P 1750 3200
-F 0 "#PWR0107" H 1750 2950 50  0001 C CNN
+F 0 "#PWR037" H 1750 2950 50  0001 C CNN
 F 1 "GND" V 1755 3072 50  0000 R CNN
 F 2 "" H 1750 3200 50  0001 C CNN
@@
 	1750 3200 1900 3200
 $Comp
-L power:GND #PWR0108
+L power:GND #PWR039
 U 1 1 5DDEE142
 P 1750 5250
-F 0 "#PWR0108" H 1750 5000 50  0001 C CNN
+F 0 "#PWR039" H 1750 5000 50  0001 C CNN
 F 1 "GND" V 1755 5122 50  0000 R CNN
 F 2 "" H 1750 5250 50  0001 C CNN
@@
 P 5150 3300
 AR Path="/5E0643C1" Ref="J?"  Part="1"
-AR Path="/5DDEBCF4/5E0643C1" Ref="J4"  Part="1"
-F 0 "J4" H 5122 3324 50  0000 R CNN
+AR Path="/5DDEBCF4/5E0643C1" Ref="J6"  Part="1"
+F 0 "J6" H 5122 3324 50  0000 R CNN
 F 1 "TO_OUTPUTS" H 5122 3233 50  0000 R CNN
 F 2 "Connector_PinHeader_2.54mm:PinHeader_1x17_P2.54mm_Vertical" H 5150 3300 50  0001 C CNN
@@
 	2700 5350 4700 5350
 $Comp
-L power:GND #PWR016
+L power:GND #PWR044
 U 1 1 5E07C333
 P 4750 2500
-F 0 "#PWR016" H 4750 2250 50  0001 C CNN
+F 0 "#PWR044" H 4750 2250 50  0001 C CNN
 F 1 "GND" V 4755 2372 50  0000 R CNN
 F 2 "" H 4750 2500 50  0001 C CNN
