File: megasequencer/brain/brain/file5E353BDC.sch (KiCad schematic (older format))
At the start: 32 parts, among them SW10 POS_7_SW, SW11 POS_8_SW, SW12 POS_9_SW, SW13 POS_10_SW, SW14 POS_11_SW, SW15 POS_12_SW, SW16 POS_13_SW, SW17 POS_14_SW, SW18 POS_15_SW, SW3 POS_0_SW, SW4 POS_1_SW, SW5 POS_2_SW, SW6 POS_3_SW, SW7 POS_4_SW, SW8 POS_5_SW, SW9 POS_6_SW

Commit message: Finish interface and continue with brain
Other:
- note added: "Resistor values for the switches:\n01: 91k\n02: 51k\n03: 36k\n04: 27k\n05: 20k\n06: 15k\n07: 12k\n08: 9k1\n09: 7k5\n10: 5k6\n11: 4k3\n12: 3k1\n13: 2k2\n14: 1k5\n15: 620"
Changed lines of the file:
@@
 Text HLabel 2800 1000 2    50   Output ~ 0
 INT_POS_5V
+Text Notes 3875 2450 0    50   ~ 0
+Resistor values for the switches:\n01: 91k\n02: 51k\n03: 36k\n04: 27k\n05: 20k\n06: 15k\n07: 12k\n08: 9k1\n09: 7k5\n10: 5k6\n11: 4k3\n12: 3k1\n13: 2k2\n14: 1k5\n15: 620
 $EndSCHEMATC
