File: megasequencer/brain/brain/brain.kicad_pcb (KiCad board)
At the start: 2 copper layers, 50 parts, among them J2 INT_CLOCK_OUT, J3 DIR_IN, J4 RESET_IN, J5 EXT_RATE_CV, J6 ZERO_IN, J7 EXT_CLOCK_IN, J8 EXT_POS_CV, U1 ATmega328P-PU, U2 TL074

Commit message: Add pwr, more inputs and outputs
Other:
- board outline added: 99.1 x 99.1 mm
Changed lines of the file:
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@@
   (general
     (thickness 1.6)
-    (drawings 0)
+    (drawings 4)
     (tracks 0)
     (zones 0)
@@
     )
   )
+  (gr_line (start 25.4 124.46) (end 25.4 25.4) (layer Edge.Cuts) (width 0.15))
+  (gr_line (start 124.46 124.46) (end 25.4 124.46) (layer Edge.Cuts) (width 0.15))
+  (gr_line (start 124.46 25.4) (end 124.46 124.46) (layer Edge.Cuts) (width 0.15))
+  (gr_line (start 25.4 25.4) (end 124.46 25.4) (layer Edge.Cuts) (width 0.15))
 )

Commit message: Fiddling with PCB a bit
Parts:
- added C1: .1uF, Capacitor_THT:C_Disc_D3.0mm_W1.6mm_P2.50mm, F.Cu at (254.6, 112.8)
- added C2: .1uF, Capacitor_THT:C_Disc_D3.0mm_W1.6mm_P2.50mm, F.Cu at (254.6, 117.1)
- added C3: .1uF, Capacitor_THT:C_Disc_D3.0mm_W1.6mm_P2.50mm, F.Cu at (254.6, 115.0)
- added C4: .1uF, Capacitor_THT:C_Disc_D3.0mm_W1.6mm_P2.50mm, F.Cu at (236.9, 135.1)
- added C5: 10uF, Capacitor_THT:CP_Radial_D5.0mm_P2.00mm, F.Cu at (274.6, 144.5)
- added C6: 10uF, Capacitor_THT:CP_Radial_D5.0mm_P2.00mm, F.Cu at (269.0, 147.3)
- added C7: 10uF, Capacitor_THT:CP_Radial_D5.0mm_P2.00mm, F.Cu at (259.4, 149.4)
- added C8: 10uF, Capacitor_THT:CP_Radial_D5.0mm_P2.00mm, F.Cu at (237.5, 142.3)
- added C9: 10uF, Capacitor_THT:CP_Radial_D5.0mm_P2.00mm, F.Cu at (243.1, 142.3)
- added D11: D_Schottky, Diode_THT:D_DO-34_SOD68_P7.62mm_Horizontal, F.Cu at (246.6, 129.9)
- added D12: D_Schottky, Diode_THT:D_DO-34_SOD68_P7.62mm_Horizontal, F.Cu at (236.8, 133.0)
- added J10: STEP_OUT, Connector_Audio:Jack_3.5mm_QingPu_WQP-PJ398SM_Vertical_CircularHoles, F.Cu at (268.0, 113.4)
- added J9: EXT_RATE_CV, Connector_Audio:Jack_3.5mm_QingPu_WQP-PJ398SM_Vertical_CircularHoles, F.Cu at (220.9, 113.4)
- added R34: 1K, Resistor_THT:R_Axial_DIN0207_L6.3mm_D2.5mm_P7.62mm_Horizontal, F.Cu at (236.9, 127.3)
- added R35: 100K, Resistor_THT:R_Axial_DIN0207_L6.3mm_D2.5mm_P7.62mm_Horizontal, F.Cu at (246.6, 127.3)
- added R36: 100K, Resistor_THT:R_Axial_DIN0207_L6.3mm_D2.5mm_P7.62mm_Horizontal, F.Cu at (236.9, 130.4)
- added R37: 100K, Resistor_THT:R_Axial_DIN0207_L6.3mm_D2.5mm_P7.62mm_Horizontal, F.Cu at (217.0, 128.2)
- added R38: 100K, Resistor_THT:R_Axial_DIN0207_L6.3mm_D2.5mm_P7.62mm_Horizontal, F.Cu at (217.0, 134.3)
- added R39: 100K, Resistor_THT:R_Axial_DIN0207_L6.3mm_D2.5mm_P7.62mm_Horizontal, F.Cu at (217.0, 131.2)
- added R40: 1K, Resistor_THT:R_Axial_DIN0207_L6.3mm_D2.5mm_P7.62mm_Horizontal, F.Cu at (274.1, 113.3)
- added R41: R, Resistor_THT:R_Axial_DIN0204_L3.6mm_D1.6mm_P7.62mm_Horizontal, F.Cu at (258.5, 145.6)
- added R42: R, Resistor_THT:R_Axial_DIN0204_L3.6mm_D1.6mm_P7.62mm_Horizontal, F.Cu at (269.1, 140.6)
- added RV5: RATE_IN_OFFSET, Potentiometer_THT:Potentiometer_Alps_RK09L_Single_Vertical, F.Cu at (227.1, 121.3)
- added RV6: RATE_IN_ATT, Potentiometer_THT:Potentiometer_Alps_RK09L_Single_Vertical, F.Cu at (240.9, 121.3)
- added U3: TL074, Package_DIP:DIP-8_W7.62mm, F.Cu at (227.1, 127.4)
- added U4: 78L05, Package_TO_SOT_THT:TO-220-3_Vertical, F.Cu at (260.3, 143.0)
- added U5: 74HC595, Package_DIP:DIP-16_W7.62mm, F.Cu at (217.0, 141.1)
- added U6: 74HC595, Package_DIP:DIP-16_W7.62mm, F.Cu at (226.9, 141.1)
- moved RV4 121.0 mm to (92.7, 69.8), turned to 90 degrees
- moved RV2 119.3 mm to (62.2, 69.8), turned to 90 degrees
- moved J7 105.2 mm to (31.8, 40.6)
- moved J6 104.9 mm to (31.8, 55.9)
- moved J4 98.2 mm to (31.8, 71.1)
- moved J3 98.1 mm to (31.8, 86.4)
- moved RV3 94.7 mm to (108.0, 69.8), turned to 90 degrees
- moved RV1 92.8 mm to (108.0, 86.4), turned to 90 degrees
- moved U1 70.5 mm to (91.4, 135.9)
- moved J8 22.7 mm to (158.8, 69.8)
Connections:
- D6 pad 2: /Analog Inputs/POS_5V -> /MC/EXT_POS_5V
- D7 pad 1: /Analog Inputs/POS_5V -> /MC/EXT_POS_5V
- R21 pad 1: /Analog Inputs/POS_5V -> /MC/EXT_POS_5V
- U1 pad 26: /MC/A3 -> /Analog Inputs/PULSE_LENGTH_5V

Commit message: Split brain into brain and interface pcbs, so everything fits
Parts:
- J9: value EXT_RATE_CV -> PULSE_LENGTH_CV
- RV4: value RATE_IN_ATT -> EXT_POS_IN_ATT
- RV5: value RATE_IN_OFFSET -> PULSE_LENGTH_IN_OFFSET
- RV6: value RATE_IN_ATT -> PULSE_LENGTH_IN_ATT
Connections:
- net /MC/D1-TX renamed /MC/PULSE_OUT
- net Net-(U5-Pad1) renamed /OUTPUTS/OUT2
- net Net-(U5-Pad15) renamed /OUTPUTS/OUT1
- net Net-(U5-Pad2) renamed /OUTPUTS/OUT3
- net Net-(U5-Pad3) renamed /OUTPUTS/OUT4
- net Net-(U5-Pad4) renamed /OUTPUTS/OUT5
- net Net-(U5-Pad5) renamed /OUTPUTS/OUT6
- net Net-(U5-Pad6) renamed /OUTPUTS/OUT7
- net Net-(U5-Pad7) renamed /OUTPUTS/OUT8
- net Net-(U6-Pad1) renamed /OUTPUTS/OUT10
- net Net-(U6-Pad15) renamed /OUTPUTS/OUT9
- net Net-(U6-Pad2) renamed /OUTPUTS/OUT11
- net Net-(U6-Pad3) renamed /OUTPUTS/OUT12
- net Net-(U6-Pad4) renamed /OUTPUTS/OUT13
- net Net-(U6-Pad5) renamed /OUTPUTS/OUT14
- net Net-(U6-Pad6) renamed /OUTPUTS/OUT15
- net Net-(U6-Pad7) renamed /OUTPUTS/OUT16
- C6 pad 1: Net-(C6-Pad1) -> Net-(C5-Pad2)
- U1 pad 11: /MC/D5 -> /OUTPUTS/SERIAL
- U1 pad 12: /MC/D6 -> /OUTPUTS/SHIFT
- U1 pad 6: /MC/D4 -> /OUTPUTS/LATCH

Commit message: Brain seem ok now, also start charting the program
Parts:
- removed J10: STEP_OUT, Connector_Audio:Jack_3.5mm_QingPu_WQP-PJ398SM_Vertical_CircularHoles
- removed J8: EXT_POS_CV, Connector_Audio:Jack_3.5mm_QingPu_WQP-PJ398SM_Vertical_CircularHoles
- removed J9: PULSE_LENGTH_CV, Connector_Audio:Jack_3.5mm_QingPu_WQP-PJ398SM_Vertical_CircularHoles
- removed the R10 at (165.2, 122.6)
- removed the R11 at (184.7, 107.4)
- removed the R12 at (165.2, 119.6)
- removed the R13 at (165.2, 116.5)
- removed the R14 at (184.7, 110.4)
- removed the R15 at (175.0, 110.4)
- removed the R2 at (175.0, 119.6)
- removed the R3 at (175.0, 122.6)
- removed the R4 at (184.7, 113.5)
- removed R40: 1K, Resistor_THT:R_Axial_DIN0207_L6.3mm_D2.5mm_P7.62mm_Horizontal
- removed the R5 at (175.0, 113.5)
- removed the R6 at (184.7, 116.5)
- removed the R7 at (129.1, 122.2)
- removed the R8 at (139.2, 110.4)
- removed the R9 at (139.2, 107.4)
- removed RV1: RATE_IN_OFFSET, Potentiometer_THT:Potentiometer_Alps_RK09L_Single_Vertical
- removed RV2: EXT_POS_IN_OFFSET, Potentiometer_THT:Potentiometer_Alps_RK09L_Single_Vertical
- removed RV3: RATE_IN_ATT, Potentiometer_THT:Potentiometer_Alps_RK09L_Single_Vertical
- removed RV4: EXT_POS_IN_ATT, Potentiometer_THT:Potentiometer_Alps_RK09L_Single_Vertical
- removed RV5: PULSE_LENGTH_IN_OFFSET, Potentiometer_THT:Potentiometer_Alps_RK09L_Single_Vertical
- removed RV6: PULSE_LENGTH_IN_ATT, Potentiometer_THT:Potentiometer_Alps_RK09L_Single_Vertical
- added C10: .1uF, Capacitor_THT:C_Disc_D3.0mm_W1.6mm_P2.50mm, F.Cu at (295.9, 21.6)
- added C11: .1uF, Capacitor_THT:C_Disc_D3.0mm_W1.6mm_P2.50mm, F.Cu at (317.4, 12.3)
- added C12: .1uF, Capacitor_THT:C_Disc_D3.0mm_W1.6mm_P2.50mm, F.Cu at (322.3, 4.24)
- added C13: .1uF, Capacitor_THT:C_Disc_D3.0mm_W1.6mm_P2.50mm, F.Cu at (301.6, 21.6)
- added J1: TOP, Connector_PinHeader_2.54mm:PinHeader_1x16_P2.54mm_Vertical, F.Cu at (275.1, -56.9)
- added R20: 100K, Resistor_THT:R_Axial_DIN0207_L6.3mm_D2.5mm_P7.62mm_Horizontal, F.Cu at (296.1, 9.89)
- added R21: 100K, Resistor_THT:R_Axial_DIN0207_L6.3mm_D2.5mm_P7.62mm_Horizontal, F.Cu at (311.5, -7.46)
- added R22: 100K, Resistor_THT:R_Axial_DIN0207_L6.3mm_D2.5mm_P7.62mm_Horizontal, F.Cu at (300.7, -3.41)
- added R23: 100K, Resistor_THT:R_Axial_DIN0207_L6.3mm_D2.5mm_P7.62mm_Horizontal, F.Cu at (274.4, 11.9)
- added R24: 100K, Resistor_THT:R_Axial_DIN0207_L6.3mm_D2.5mm_P7.62mm_Horizontal, F.Cu at (285.1, 16.0)
- added R25: 100K, Resistor_THT:R_Axial_DIN0207_L6.3mm_D2.5mm_P7.62mm_Horizontal, F.Cu at (300.7, 0.64)
- added R26: 100K, Resistor_THT:R_Axial_DIN0207_L6.3mm_D2.5mm_P7.62mm_Horizontal, F.Cu at (295.9, 13.9)
- added R27: 100K, Resistor_THT:R_Axial_DIN0207_L6.3mm_D2.5mm_P7.62mm_Horizontal, F.Cu at (311.5, -3.41)
- added R34: 100K, Resistor_THT:R_Axial_DIN0207_L6.3mm_D2.5mm_P7.62mm_Horizontal, F.Cu at (322.3, -3.41)
- added R35: 100K, Resistor_THT:R_Axial_DIN0207_L6.3mm_D2.5mm_P7.62mm_Horizontal, F.Cu at (317.6, 8.74)
- added R36: 100K, Resistor_THT:R_Axial_DIN0207_L6.3mm_D2.5mm_P7.62mm_Horizontal, F.Cu at (322.3, 0.64)
- added R37: 100K, Resistor_THT:R_Axial_DIN0207_L6.3mm_D2.5mm_P7.62mm_Horizontal, F.Cu at (285.1, 20.0)
- added U7: TL074, Package_DIP:DIP-14_W7.62mm, F.Cu at (285.3, -7.41)
- added U8: TL074, Package_DIP:DIP-14_W7.62mm, F.Cu at (274.4, -7.41)
- D1, D2: value D_Schottky -> S
- D3: renamed from D6; value D_Schottky -> S
- D4: renamed from D7; value D_Schottky -> S
- D5: renamed from D11; value D_Schottky -> S
- D6: renamed from D12; value D_Schottky -> S
- J2: value INT_CLOCK_OUT -> BOTTOM; footprint Connector_Audio:Jack_3.5mm_QingPu_WQP-PJ398SM_Vertical_CircularHoles -> Connector_PinHeader_2.54mm:PinHeader_1x16_P2.54mm_Vertical
- J3: value DIR_IN -> Keyboard; footprint Connector_Audio:Jack_3.5mm_QingPu_WQP-PJ398SM_Vertical_CircularHoles -> Connector_PinHeader_2.54mm:PinHeader_1x02_P2.54mm_Vertical
- J4: value RESET_IN -> EURO_PWR_2x5; footprint Connector_Audio:Jack_3.5mm_QingPu_WQP-PJ398SM_Vertical_CircularHoles -> Connector_PinHeader_2.54mm:PinHeader_2x05_P2.54mm_Vertical
- J5: value EXT_RATE_CV -> ICSP; footprint Connector_Audio:Jack_3.5mm_QingPu_WQP-PJ398SM_Vertical_CircularHoles -> Connector_PinHeader_2.54mm:PinHeader_2x05_P2.54mm_Vertical
- J6: value ZERO_IN -> TO_OUTPUTS; footprint Connector_Audio:Jack_3.5mm_QingPu_WQP-PJ398SM_Vertical_CircularHoles -> Connector_PinHeader_2.54mm:PinHeader_1x17_P2.54mm_Vertical
- J7: value EXT_CLOCK_IN -> FROM_OUTPUTS; footprint Connector_Audio:Jack_3.5mm_QingPu_WQP-PJ398SM_Vertical_CircularHoles -> Connector_PinHeader_2.54mm:PinHeader_1x06_P2.54mm_Vertical
- R1: value 91K -> 10K
- R16: value 2K2 -> 1K
- R17: value 1K5 -> 1K
- R18: value 620 -> 1K
- R19: value 10K -> 1K
- R28, R29: value 10K -> 100K
- U4: renamed from U3; value TL074 -> TL072
- moved J6 348.1 mm to (361.1, -56.9)
- moved J4 338.7 mm to (361.1, -8.27)
- moved J3 299.8 mm to (295.2, -56.9)
- moved J7 269.3 mm to (296.8, -7.16)
- moved J2 220.3 mm to (279.8, -56.9)
- moved J5 213.5 mm to (390.9, -8.27)
- moved R29 206.0 mm to (311.5, 0.64)
- moved R1 204.9 mm to (283.7, -57.1)
- moved R28 199.3 mm to (306.8, 8.74)
- moved R19 177.6 mm to (300.7, -7.46)
- moved R16 157.2 mm to (285.1, 11.9)
- moved R39 151.7 mm to (300.7, 4.69)
- moved R32 147.2 mm to (322.3, -7.46)
- moved R38 146.9 mm to (306.7, 18.0)
- moved R18 141.7 mm to (274.4, 20.0)
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- renumbered C5 to C1, C6 to C2, C7 to C3, C1 to C4, C2 to C5, C3 to C6, C4 to C7, R24 to R10, R25 to R11, R36 to R12, R26 to R13, R27 to R14, R37 to R15, R41 to R2, R42 to R3, R20 to R4, R21 to R5, R34 to R6, R22 to R7, R23 to R8, R35 to R9, U4 to U1, U1 to U2, U2 to U3
Connections:
- C1 pad 2: Net-(C5-Pad2) -> Net-(C1-Pad2)
- C2 pad 1: Net-(C5-Pad2) -> Net-(C1-Pad2)
- C3 pad 2: Net-(C5-Pad2) -> Net-(C1-Pad2)
- R1 pad 1: Net-(R1-Pad1) -> /MC/INT_POS_5V
- R1 pad 2: /Keyboard/INT_POS_5V -> GND
- R13 pad 2: Net-(R26-Pad2) -> /EXT_POS_A
- R14 pad 2: Net-(R27-Pad2) (its old number) -> /EXT_POS_A
- R15 pad 2: Net-(R37-Pad2) -> /PULSELEN_A
- R16 pad 1: Net-(R16-Pad1) -> /OFFSET_A
- R16 pad 2: /Keyboard/INT_POS_5V -> Net-(R16-Pad2)
- R17 pad 1: Net-(R17-Pad1) -> /OUTPUT_B
- R17 pad 2: /Keyboard/INT_POS_5V -> Net-(R17-Pad2)
- R18 pad 1: Net-(R18-Pad1) -> /OUTPUT_C
- R18 pad 2: /Keyboard/INT_POS_5V -> Net-(R18-Pad2)
- R19 pad 1: /Keyboard/INT_POS_5V -> /OUTPUT_D
- R19 pad 2: GND -> Net-(R19-Pad2)
- R2 pad 2: Net-(J1-Pad1) -> Net-(J4-Pad1)
- R28 pad 1: GND -> Net-(R26-Pad2)
- R28 pad 2: Net-(D9-Pad2) -> Net-(R28-Pad2)
- R29 pad 1: GND -> Net-(R24-Pad2)
- R29 pad 2: Net-(D10-Pad2) -> Net-(R29-Pad2)
- R3 pad 2: Net-(J1-Pad10) -> Net-(J4-Pad10)
- R30 pad 2: Net-(R26-Pad2) -> Net-(R30-Pad2)
- R31 pad 2: Net-(R27-Pad2) (its old number) -> Net-(R31-Pad2)
- R32 pad 1: Net-(R26-Pad2) -> Net-(R28-Pad2)
- R32 pad 2: Net-(R32-Pad2) -> Net-(J7-Pad1)
- R33 pad 1: Net-(R27-Pad2) (its old number) -> Net-(R28-Pad2)
- R33 pad 2: Net-(R33-Pad2) -> /OFFSET_A
- R38 pad 1: Net-(R38-Pad1) -> Net-(R31-Pad2)
- R38 pad 2: Net-(R37-Pad2) -> Net-(J7-Pad4)
- R39 pad 1: Net-(R37-Pad2) -> Net-(R31-Pad2)
- R39 pad 2: Net-(R39-Pad2) -> /OFFSET_D
- U1 pad 2: Net-(C5-Pad2) -> Net-(C1-Pad2)
- U2 pad 14: /Digital IO/SEQ_DIR -> /SEQ_DIR_D
- U2 pad 15: /Digital IO/INT_CLOCK -> /INT_CLOCK_D
- U2 pad 16: /Digital IO/SEQ_ZERO -> /SEQ_ZERO_D
- U2 pad 25: /Keyboard/INT_POS_5V -> /MC/INT_POS_5V
- U2 pad 3: /MC/PULSE_OUT -> /STEP_PULSE_D
- U2 pad 4: /Digital IO/EXT_CLOCK -> /EXT_CLOCK_D
- U2 pad 5: /Digital IO/SEQ_RESET -> /SEQ_RESET_D
- U3 pad 2: Net-(R26-Pad2) -> /EXT_POS_A
- U3 pad 9: Net-(R27-Pad2) (its old number) -> /EXT_POS_A
- U4 pad 2: Net-(R37-Pad2) -> /PULSELEN_A
- U5 pad 1: /OUTPUTS/OUT2 -> Net-(J6-Pad3)
- U5 pad 15: /OUTPUTS/OUT1 -> Net-(J6-Pad2)
- U5 pad 2: /OUTPUTS/OUT3 -> Net-(J6-Pad4)
- U5 pad 3: /OUTPUTS/OUT4 -> Net-(J6-Pad5)
- U5 pad 4: /OUTPUTS/OUT5 -> Net-(J6-Pad6)
- U5 pad 5: /OUTPUTS/OUT6 -> Net-(J6-Pad7)
- U5 pad 6: /OUTPUTS/OUT7 -> Net-(J6-Pad8)
- U5 pad 7: /OUTPUTS/OUT8 -> Net-(J6-Pad9)
- U6 pad 1: /OUTPUTS/OUT10 -> Net-(J6-Pad11)
- U6 pad 15: /OUTPUTS/OUT9 -> Net-(J6-Pad10)
- U6 pad 2: /OUTPUTS/OUT11 -> Net-(J6-Pad12)
- U6 pad 3: /OUTPUTS/OUT12 -> Net-(J6-Pad13)
- U6 pad 4: /OUTPUTS/OUT13 -> Net-(J6-Pad14)
- U6 pad 5: /OUTPUTS/OUT14 -> Net-(J6-Pad15)
- U6 pad 6: /OUTPUTS/OUT15 -> Net-(J6-Pad16)
- U6 pad 7: /OUTPUTS/OUT16 -> Net-(J6-Pad17)

Commit message: Almost done now with both pcbs
Parts:
- added C14: 22pF, Capacitor_THT:C_Disc_D3.0mm_W1.6mm_P2.50mm, F.Cu at (49.5, 92.7)
- added C15: 22pF, Capacitor_THT:C_Disc_D3.0mm_W1.6mm_P2.50mm, F.Cu at (49.5, 102.9)
- added C16: 15pF, Capacitor_THT:C_Disc_D3.0mm_W1.6mm_P2.50mm, F.Cu at (57.1, 90.2)
- added C17: 100nF, Capacitor_THT:C_Disc_D3.0mm_W1.6mm_P2.50mm, F.Cu at (70.1, 90.4)
- added C18: 100nF, Capacitor_THT:C_Disc_D3.0mm_W1.6mm_P2.50mm, F.Cu at (59.7, 69.2)
- added D7: 1N4148, Diode_THT:D_A-405_P7.62mm_Horizontal, F.Cu at (47.0, 81.3)
- added FB1: Ferrite_Bead, Inductor_THT:L_Axial_L6.6mm_D2.7mm_P10.16mm_Horizontal_Vishay_IM-2, F.Cu at (67.3, 114.3)
- added FB2: Ferrite_Bead, Inductor_THT:L_Axial_L6.6mm_D2.7mm_P10.16mm_Horizontal_Vishay_IM-2, F.Cu at (57.1, 109.2)
- added H1: M3, MountingHole:MountingHole_3.2mm_M3_Pad, F.Cu at (29.2, 29.2)
- added H2: M3, MountingHole:MountingHole_3.2mm_M3_Pad, F.Cu at (29.2, 120.7)
- added H3: M3, MountingHole:MountingHole_3.2mm_M3_Pad, F.Cu at (120.7, 29.2)
- added H4: M3, MountingHole:MountingHole_3.2mm_M3_Pad, F.Cu at (120.7, 120.7)
- added J8: RIGHT, Connector_PinSocket_2.54mm:PinSocket_1x04_P2.54mm_Vertical, F.Cu at (122.4, 73.7)
- added R40: 330, Resistor_THT:R_Axial_DIN0207_L6.3mm_D2.5mm_P7.62mm_Horizontal, F.Cu at (54.6, 73.7)
- added R41: 10K, Resistor_THT:R_Axial_DIN0207_L6.3mm_D2.5mm_P7.62mm_Horizontal, F.Cu at (54.6, 77.5)
- added SW1: RST, Button_Switch_THT:SW_PUSH_6mm, B.Cu at (54.0, 64.8)
- added Y1: Crystal, Crystal:Crystal_HC18-U_Vertical, F.Cu at (54.6, 95.2)
- C1, C2, C3, C8, C9, J3, J4, J5, J6, J7: moved to B.Cu
- J1: footprint Connector_PinHeader_2.54mm:PinHeader_1x16_P2.54mm_Vertical -> Connector_PinSocket_2.54mm:PinSocket_1x16_P2.54mm_Vertical
- J2: footprint Connector_PinHeader_2.54mm:PinHeader_1x16_P2.54mm_Vertical -> Connector_PinSocket_2.54mm:PinSocket_1x08_P2.54mm_Vertical
- R2, R3: value R -> 10
- U1: footprint Package_TO_SOT_THT:TO-220-3_Vertical -> Package_TO_SOT_THT:TO-220-3_Horizontal_TabDown
- moved J6 356.1 mm to (29.2, 72.4), turned to 180 degrees
- moved J5 337.3 mm to (78.7, 119.4), turned to 270 degrees
- moved J4 291.4 mm to (99.1, 119.4), turned to 270 degrees
- moved R32 290.9 mm to (35.6, 41.9), turned to 270 degrees
- moved J2 288.5 mm to (53.3, 121.9), turned to 270 degrees
- moved R34 282.7 mm to (43.2, 41.9), turned to 270 degrees
- moved R35 276.1 mm to (43.2, 39.4), turned to 90 degrees
- moved R36 274.6 mm to (50.8, 41.9), turned to 270 degrees
- moved J7 273.4 mm to (29.2, 48.9)
- moved R33 272.3 mm to (35.6, 39.4), turned to 90 degrees
- moved R21 261.6 mm to (54.6, 41.9), turned to 270 degrees
- moved J3 260.6 mm to (71.1, 76.2)
- moved R20 258.7 mm to (39.4, 41.9), turned to 270 degrees
- moved R22 257.7 mm to (47.0, 41.9), turned to 270 degrees
- moved R1 252.8 mm to (71.1, 79.8), turned to 270 degrees
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Connections:
- C1 pad 2: Net-(C1-Pad2) -> GND
- C2 pad 1: Net-(C1-Pad2) -> GND
- C3 pad 2: Net-(C1-Pad2) -> GND
- J1 pad 14: /OFFSET_A -> /OUTPUT_A
- J1 pad 6: /OUTPUT_E -> /OUTPUT_F
- J2 pad 4: Net-(J2-Pad4) -> /SEQ_RESET_D
- J2 pad 5: Net-(J2-Pad5) -> /SEQ_ZERO_D
- J2 pad 6: Net-(J2-Pad6) -> /SEQ_DIR_D
- J2 pad 7: Net-(J2-Pad7) -> +5V
- J2 pad 8: Net-(J2-Pad8) -> GND
- J4 pad 4: Net-(C1-Pad2) -> GND
- J4 pad 6: Net-(C1-Pad2) -> GND
- J4 pad 8: Net-(C1-Pad2) -> GND
- J7 pad 6: /OUTPUT_E -> /OUTPUT_F
- R13 pad 2: /EXT_POS_A -> /EXT_RATE_A
- R16 pad 1: /OFFSET_A -> /OUTPUT_A
- U1 pad 2: Net-(C1-Pad2) -> GND
- U2 pad 13: /MC/D7 -> /SEQ_DIR_D
- U2 pad 14: /SEQ_DIR_D -> /SEQ_ZERO_D
- U2 pad 15: /INT_CLOCK_D -> /MC/D9
- U2 pad 16: /SEQ_ZERO_D -> /MC/D10
- U2 pad 2: /MC/D0-RX -> /INT_CLOCK_D
- U2 pad 20: +5V -> Net-(C17-Pad2)
- U2 pad 23: /Analog Inputs/RATE_5V -> /MC/EXT_POS_5V
- U2 pad 24: /MC/EXT_POS_5V -> /Analog Inputs/RATE_5V
- U2 pad 7: +5V -> Net-(C16-Pad2)
- U3 pad 13: Net-(R10-Pad1) -> /EXT_POS_A
- U3 pad 14: Net-(R5-Pad2) -> Net-(R10-Pad2)
- U3 pad 2: /EXT_POS_A -> /EXT_RATE_A
- U3 pad 8: Net-(R10-Pad2) -> Net-(R5-Pad2)
- U3 pad 9: /EXT_POS_A -> Net-(R10-Pad1)
Routing:
- net +5V: track 0.00 -> 211.7 mm
- net +12V: track 0.00 -> 124.7 mm
- net Net-(R28-Pad2): track 0.00 -> 124.4 mm
- net -12V: track 0.00 -> 122.9 mm
- net Net-(R16-Pad2): track 0.00 -> 101.8 mm
- net Net-(R20-Pad2): track 0.00 -> 81.2 mm
- net Net-(R29-Pad2): track 0.00 -> 79.2 mm
- net /MC/RST: track 0.00 -> 72.4 mm
- net Net-(R22-Pad2): track 0.00 -> 69.0 mm
- net Net-(R17-Pad2): track 0.00 -> 60.8 mm
- net /SEQ_RESET_D: track 0.00 -> 59.3 mm
- net /OUTPUTS/SHIFT: track 0.00 -> 57.3 mm
- net /OUTPUTS/LATCH: track 0.00 -> 56.2 mm
- net /EXT_CLOCK_D: track 0.00 -> 54.6 mm
- net /STEP_PULSE_D: track 0.00 -> 53.2 mm
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- added copper zone on B.Cu, net GND
- added copper zone on F.Cu, net GND
Other:
- board text added: "-12V"
- board text added: "1"
