File: megasequencer/brain/brain/brain.sch (KiCad schematic (older format))
At the start: 0 parts

Commit message: Split brain into brain and interface pcbs, so everything fits
Parts:
- added J11: ROWA, symbol Connector_Generic:Conn_01x32
Connections:
- net labels added: GND
- wire segments 13 -> 61
Changed lines of the file:
@@
 Mega Sequencer Brain
 $Sheet
-S 600  1400 650  150
+S 3100 900  650  150
 U 5E3019D8
 F0 "Power" 50
@@
 $EndSheet
 $Sheet
-S 600  3000 650  200
+S 3100 2500 650  200
 U 5E353BDD
 F0 "Keyboard" 50
 F1 "file5E353BDC.sch" 50
-F2 "INT_POS_5V" O R 1250 3100 50
-$EndSheet
-$Sheet
-S 2750 2350 750  4100
+F2 "INT_POS_5V" O R 3750 2600 50
+$EndSheet
+$Sheet
+S 5250 1850 750  4100
 U 5E366867
 F0 "MC" 50
 F1 "file5E366866.sch" 50
-F2 "RATE_5V" I L 2750 2450 50
-F3 "EXT_POS_5V" I L 2750 2550 50
-F4 "INT_POS_5V" I L 2750 3100 50
-F5 "SEQ_CLOCK" I L 2750 3950 50
-F6 "SEQ_RESET" I L 2750 3750 50
-F7 "SEQ_DIR" I L 2750 3650 50
-F8 "INT_CLOCK" O L 2750 3550 50
-F9 "SEQ_ZERO" I L 2750 3850 50
-F10 "PULSE_LENGTH_5V" I L 2750 2650 50
-F11 "PULSE_OUT" O L 2750 4050 50
-F12 "STEPS_DATA" O L 2750 4800 50
-F13 "STEPS_CLOCK" O L 2750 4900 50
-F14 "STEPS_LATCH" O L 2750 5000 50
-$EndSheet
-$Sheet
-S 600  2400 650  450
+F2 "RATE_5V" I L 5250 1950 50
+F3 "EXT_POS_5V" I L 5250 2050 50
+F4 "INT_POS_5V" I L 5250 2600 50
+F5 "SEQ_CLOCK" I L 5250 3450 50
+F6 "SEQ_RESET" I L 5250 3250 50
+F7 "SEQ_DIR" I L 5250 3150 50
+F8 "INT_CLOCK" O L 5250 3050 50
+F9 "SEQ_ZERO" I L 5250 3350 50
+F10 "PULSE_LENGTH_5V" I L 5250 2150 50
+F11 "PULSE_OUT" O L 5250 3550 50
+F12 "STEPS_DATA" O L 5250 4300 50
+F13 "STEPS_CLOCK" O L 5250 4400 50
+F14 "STEPS_LATCH" O L 5250 4500 50
+$EndSheet
+$Sheet
+S 3100 1900 650  450
 U 5E36D63E
 F0 "Analog Inputs" 50
 F1 "file5E36D63D.sch" 50
-F2 "RATE_5V" I R 1250 2450 50
-F3 "POS_5V" O R 1250 2550 50
-F4 "PULSE_LENGTH_5V" O R 1250 2650 50
-$EndSheet
-Wire Wire Line
-	1250 2450 2750 2450
-Wire Wire Line
-	1250 2550 2750 2550
-Wire Wire Line
-	1250 3100 2750 3100
-$Sheet
-S 600  3450 650  1000
+F2 "RATE_5V" I R 3750 1950 50
+F3 "POS_5V" O R 3750 2050 50
+F4 "PULSE_LENGTH_5V" O R 3750 2150 50
+$EndSheet
+Wire Wire Line
+	3750 1950 5250 1950
+Wire Wire Line
+	3750 2050 5250 2050
+Wire Wire Line
+	3750 2600 5250 2600
+$Sheet
+S 3100 2950 650  1000
 U 5DDA0F22
 F0 "Digital IO" 50
 F1 "file5DDA0F21.sch" 50
-F2 "INT_CLOCK" I R 1250 3550 50
-F3 "SEQ_DIR" O R 1250 3650 50
-F4 "SEQ_RESET" O R 1250 3750 50
-F5 "SEQ_ZERO" O R 1250 3850 50
-F6 "EXT_CLOCK" O R 1250 3950 50
-F7 "STEP_PULSE" I R 1250 4050 50
-$EndSheet
-Wire Wire Line
-	1250 3650 2750 3650
-Wire Wire Line
-	1250 3750 2750 3750
-Wire Wire Line
-	1250 3950 2750 3950
-Wire Wire Line
-	1250 3550 2750 3550
-Wire Wire Line
-	1250 3850 2750 3850
-Wire Wire Line
-	1250 2650 2750 2650
-$Sheet
-S 600  4700 650  900
+F2 "INT_CLOCK" I R 3750 3050 50
+F3 "SEQ_DIR" O R 3750 3150 50
+F4 "SEQ_RESET" O R 3750 3250 50
+F5 "SEQ_ZERO" O R 3750 3350 50
+F6 "EXT_CLOCK" O R 3750 3450 50
+F7 "STEP_PULSE" I R 3750 3550 50
+$EndSheet
+Wire Wire Line
+	3750 3150 5250 3150
+Wire Wire Line
+	3750 3250 5250 3250
+Wire Wire Line
+	3750 3450 5250 3450
+Wire Wire Line
+	3750 3050 5250 3050
+Wire Wire Line
+	3750 3350 5250 3350
+Wire Wire Line
+	3750 2150 5250 2150
+Wire Wire Line
+	3750 3550 5250 3550
+$Sheet
+S 3100 4200 700  1750
 U 5DDEBCF4
 F0 "OUTPUTS" 50
 F1 "file5DDEBCF3.sch" 50
-F2 "SERIAL" I R 1250 4800 50
-F3 "SHIFT" I R 1250 4900 50
-F4 "LATCH" I R 1250 5000 50
-$EndSheet
-Wire Wire Line
-	1250 4050 2750 4050
-Wire Wire Line
-	2750 4800 1250 4800
-Wire Wire Line
-	2750 4900 1250 4900
-Wire Wire Line
-	2750 5000 1250 5000
+F2 "SERIAL" I R 3800 4300 50
+F3 "SHIFT" I R 3800 4400 50
+F4 "LATCH" I R 3800 4500 50
+F5 "OUT1" O L 3100 4300 50
+F6 "OUT2" O L 3100 4400 50
+F7 "OUT3" O L 3100 4500 50
+F8 "OUT4" O L 3100 4600 50
+F9 "OUT5" O L 3100 4700 50
+F10 "OUT6" O L 3100 4800 50
+F11 "OUT7" O L 3100 4900 50
+F12 "OUT8" O L 3100 5000 50
+F13 "OUT9" O L 3100 5150 50
+F14 "OUT10" O L 3100 5250 50
+F15 "OUT11" O L 3100 5350 50
+F16 "OUT12" O L 3100 5450 50
+F17 "OUT13" O L 3100 5550 50
+F18 "OUT14" O L 3100 5650 50
+F19 "OUT15" O L 3100 5750 50
+F20 "OUT16" O L 3100 5850 50
+$EndSheet
+Wire Wire Line
+	3800 4300 5250 4300
+Wire Wire Line
+	3800 4400 5250 4400
+Wire Wire Line
+	3800 4500 5250 4500
+$Comp
+L Connector_Generic:Conn_01x32 J11
+U 1 1 5E0452B4
+P 1000 4100
+F 0 "J11" H 918 2275 50  0000 C CNN
+F 1 "ROWA" H 918 2366 50  0000 C CNN
+F 2 "" H 1000 4100 50  0001 C CNN
+F 3 "~" H 1000 4100 50  0001 C CNN
+	1    1000 4100
+	-1   0    0    1
+$EndComp
+Wire Wire Line
+	3100 5850 1200 5850
+Wire Wire Line
+	1200 5850 1200 5600
+Wire Wire Line
+	3100 5750 1250 5750
+Wire Wire Line
+	1250 5750 1250 5500
+Wire Wire Line
+	1250 5500 1200 5500
+Wire Wire Line
+	3100 5650 1300 5650
+Wire Wire Line
+	1300 5650 1300 5400
+Wire Wire Line
+	1300 5400 1200 5400
+Wire Wire Line
+	3100 5550 1350 5550
+Wire Wire Line
+	1350 5550 1350 5300
+Wire Wire Line
+	1350 5300 1200 5300
+Wire Wire Line
+	3100 5450 1400 5450
+Wire Wire Line
+	1400 5450 1400 5200
+Wire Wire Line
+	1400 5200 1200 5200
+Wire Wire Line
+	3100 5350 1450 5350
+Wire Wire Line
+	1450 5350 1450 5100
+Wire Wire Line
+	1450 5100 1200 5100
+Wire Wire Line
+	3100 5250 1500 5250
+Wire Wire Line
+	1500 5250 1500 5000
+Wire Wire Line
+	1500 5000 1200 5000
+Wire Wire Line
+	3100 5150 1550 5150
+Wire Wire Line
+	1550 5150 1550 4900
+Wire Wire Line
+	1550 4900 1200 4900
+Wire Wire Line
+	3100 5000 1600 5000
+Wire Wire Line
+	1600 5000 1600 4800
+Wire Wire Line
+	1600 4800 1200 4800
+Wire Wire Line
+	3100 4900 1650 4900
+Wire Wire Line
+	1650 4900 1650 4700
+Wire Wire Line
+	1650 4700 1200 4700
+Wire Wire Line
+	3100 4800 1700 4800
+Wire Wire Line
+	1700 4800 1700 4600
+Wire Wire Line
+	1700 4600 1200 4600
+Wire Wire Line
+	3100 4700 1750 4700
+Wire Wire Line
+	1750 4700 1750 4500
+Wire Wire Line
+	1750 4500 1200 4500
+Wire Wire Line
+	3100 4600 1800 4600
+Wire Wire Line
+	1800 4600 1800 4400
+Wire Wire Line
+	1800 4400 1200 4400
+Wire Wire Line
+	3100 4500 1850 4500
+Wire Wire Line
+	1850 4500 1850 4300
+Wire Wire Line
+	1850 4300 1200 4300
+Wire Wire Line
+	3100 4400 1900 4400
+Wire Wire Line
+	1900 4400 1900 4200
+Wire Wire Line
+	1900 4200 1200 4200
+Wire Wire Line
+	3100 4300 1950 4300
+Wire Wire Line
+	1950 4300 1950 4100
+Wire Wire Line
+	1950 4100 1200 4100
+$Comp
+L power:GND #PWR0109
+U 1 1 5E05275C
+P 1350 4000
+F 0 "#PWR0109" H 1350 3750 50  0001 C CNN
+F 1 "GND" V 1355 3872 50  0000 R CNN
+F 2 "" H 1350 4000 50  0001 C CNN
+F 3 "" H 1350 4000 50  0001 C CNN
+	1    1350 4000
+	0    -1   -1   0
+$EndComp
+Wire Wire Line
+	1200 4000 1350 4000
 $EndSCHEMATC

Commit message: Finish interface and continue with brain
Parts:
- removed J11: ROWA, symbol Connector_Generic:Conn_01x32
- added J2: Keyboard, Connector_PinHeader_2.54mm:PinHeader_1x02_P2.54mm_Vertical, symbol Connector_Generic:Conn_01x02
- added R1: 10K, Resistor_THT:R_Axial_DIN0207_L6.3mm_D2.5mm_P7.62mm_Horizontal, symbol Device:R
Connections:
- net labels added: +5V, EXT_CLOCK_D, EXT_POS_A, EXT_RATE_A, INT_CLOCK_D, PULSELEN_A, SEQ_DIR_D, SEQ_RESET_D, SEQ_ZERO_D, STEP_PULSE_D
- wire segments 61 -> 21
Other:
- note added: "Resistor values for the keyboard switches:\n01: 91k\n02: 51k\n03: 36k\n04: 27k\n05: 20k\n06: 15k\n07: 12k\n08: 9k1\n09: 7k5\n10: 5k6\n11: 4k3\n12: 3k1\n13: 2k2\n14: 1k5\n15: 620\n16: 0"

Commit message: Brain seem ok now, also start charting the program
Parts:
- added J1: TOP, Connector_PinHeader_2.54mm:PinHeader_1x16_P2.54mm_Vertical, symbol Connector_Generic:Conn_01x16
- added J2: BOTTOM, Connector_PinHeader_2.54mm:PinHeader_1x16_P2.54mm_Vertical, symbol Connector_Generic:Conn_01x16
- renumbered J2 to J3
Connections:
- net +5V: now also J2.15 (Pin_15)
- net EXT_CLOCK_D: now also J1.5 (Pin_5)
- net EXT_POS_A: now also J2.11 (Pin_11), J2.9 (Pin_9)
- net GND: now also J1.1 (Pin_1), J1.16 (Pin_16), J2.1 (Pin_1), J2.16 (Pin_16)
- net INT_CLOCK_D: now also J1.4 (Pin_4)
- net PULSELEN_A: now also J2.10 (Pin_10)
- net SEQ_DIR_D: now also J2.14 (Pin_14)
- net SEQ_RESET_D: now also J2.12 (Pin_12)
- net SEQ_ZERO_D: now also J2.13 (Pin_13)
- net STEP_PULSE_D: now also J1.3 (Pin_3)
- new net OFFSET_A: J1.14 (Pin_14), J1.15 (Pin_15)
- new net OFFSET_B: J1.13 (Pin_13)
- new net OFFSET_C: J1.11 (Pin_11)
- new net OFFSET_D: J1.9 (Pin_9)
- new net OUTPUT_B: J1.12 (Pin_12)
- new net OUTPUT_C: J1.10 (Pin_10)
- new net OUTPUT_D: J1.8 (Pin_8)
- new net OUTPUT_E: J1.6 (Pin_6), J1.7 (Pin_7)
- no-connect marks 0 -> 8
Changed lines of the file:
@@
 	9300 2775 9275 2775
 $Comp
-L power:GND #PWR05
+L power:GND #PWR06
 U 1 1 5E086E04
 P 8700 2775
-AR Path="/5E086E04" Ref="#PWR05"  Part="1"
+AR Path="/5E086E04" Ref="#PWR06"  Part="1"
 AR Path="/5E353BDD/5E086E04" Ref="#PWR?"  Part="1"
-F 0 "#PWR05" H 8700 2525 50  0001 C CNN
+F 0 "#PWR06" H 8700 2525 50  0001 C CNN
 F 1 "GND" H 8705 2602 50  0000 C CNN
 F 2 "" H 8700 2775 50  0001 C CNN
@@
 	8900 2775 8700 2775
 $Comp
-L Connector_Generic:Conn_01x02 J2
+L Connector_Generic:Conn_01x02 J3
 U 1 1 5E087A11
 P 9500 2775
-F 0 "J2" H 9580 2767 50  0000 L CNN
+F 0 "J3" H 9580 2767 50  0000 L CNN
 F 1 "Keyboard" H 9580 2676 50  0000 L CNN
 F 2 "Connector_PinHeader_2.54mm:PinHeader_1x02_P2.54mm_Vertical" H 9500 2775 50  0001 C CNN
@@
 $EndComp
 $Comp
-L power:+5V #PWR06
+L power:+5V #PWR07
 U 1 1 5E087C9A
 P 9300 2875
-F 0 "#PWR06" H 9300 2725 50  0001 C CNN
+F 0 "#PWR07" H 9300 2725 50  0001 C CNN
 F 1 "+5V" V 9315 3003 50  0000 L CNN
 F 2 "" H 9300 2875 50  0001 C CNN
@@
 STEP_PULSE_D
 $Sheet
-S 1500 2375 1000 3775
+S 8100 700  850  925
 U 5E0D4D6E
 F0 "Output Offset" 50
 F1 "output_offset.sch" 50
+F2 "AO_IN" I R 8950 825 50
+F3 "BO_IN" I R 8950 1025 50
+F4 "CO_IN" I R 8950 1225 50
+F5 "DO_IN" I R 8950 1425 50
+F6 "A_OUT" O R 8950 925 50
+F7 "B_OUT" O R 8950 1125 50
+F8 "C_OUT" O R 8950 1325 50
+F9 "D_OUT" O R 8950 1525 50
+F10 "E_OUT" O L 8100 825 50
+F11 "F_OUT" O L 8100 925 50
 $EndSheet
+Wire Wire Line
+	8950 825  8950 925
+Wire Wire Line
+	8950 825  9525 825
+Wire Wire Line
+	8950 1025 9525 1025
+Wire Wire Line
+	8950 925  9525 925
+Wire Wire Line
+	8950 1125 9525 1125
+Wire Wire Line
+	8950 1225 9525 1225
+Wire Wire Line
+	8950 1325 9525 1325
+Wire Wire Line
+	8950 1425 9525 1425
+Wire Wire Line
+	8950 1525 9525 1525
+Text Label 9525 825  2    50   ~ 0
+OFFSET_A
+Text Label 9525 1025 2    50   ~ 0
+OFFSET_B
+Text Label 9525 1225 2    50   ~ 0
+OFFSET_C
+Text Label 9525 1425 2    50   ~ 0
+OFFSET_D
+Text Label 9525 925  2    50   ~ 0
+OUTPUT_A
+Text Label 9525 1125 2    50   ~ 0
+OUTPUT_B
+Text Label 9525 1325 2    50   ~ 0
+OUTPUT_C
+Text Label 9525 1525 2    50   ~ 0
+OUTPUT_D
+$Comp
+L Connector_Generic:Conn_01x16 J1
+U 1 1 5E1623FC
+P 3250 2025
+F 0 "J1" H 3168 1000 50  0000 C CNN
+F 1 "TOP" H 3168 1091 50  0000 C CNN
+F 2 "Connector_PinHeader_2.54mm:PinHeader_1x16_P2.54mm_Vertical" H 3250 2025 50  0001 C CNN
+F 3 "~" H 3250 2025 50  0001 C CNN
+	1    3250 2025
+	-1   0    0    1
+$EndComp
+$Comp
+L Connector_Generic:Conn_01x16 J2
+U 1 1 5E162F36
+P 3250 4100
+F 0 "J2" H 3168 3075 50  0000 C CNN
+F 1 "BOTTOM" H 3168 3166 50  0000 C CNN
+F 2 "Connector_PinHeader_2.54mm:PinHeader_1x16_P2.54mm_Vertical" H 3250 4100 50  0001 C CNN
+F 3 "~" H 3250 4100 50  0001 C CNN
+	1    3250 4100
+	-1   0    0    1
+$EndComp
+$Comp
+L power:GND #PWR01
+U 1 1 5E164133
+P 3750 1225
+AR Path="/5E164133" Ref="#PWR01"  Part="1"
+AR Path="/5E353BDD/5E164133" Ref="#PWR?"  Part="1"
+F 0 "#PWR01" H 3750 975 50  0001 C CNN
+F 1 "GND" V 3755 1052 50  0000 C CNN
+F 2 "" H 3750 1225 50  0001 C CNN
+F 3 "" H 3750 1225 50  0001 C CNN
+	1    3750 1225
+	0    -1   1    0
+$EndComp
+Wire Wire Line
+	3450 1225 3750 1225
+$Comp
+L power:GND #PWR02
+U 1 1 5E165C44
+P 3750 2725
+AR Path="/5E165C44" Ref="#PWR02"  Part="1"
+AR Path="/5E353BDD/5E165C44" Ref="#PWR?"  Part="1"
+F 0 "#PWR02" H 3750 2475 50  0001 C CNN
+F 1 "GND" V 3755 2552 50  0000 C CNN
+F 2 "" H 3750 2725 50  0001 C CNN
+F 3 "" H 3750 2725 50  0001 C CNN
+	1    3750 2725
+	0    -1   1    0
+$EndComp
+Wire Wire Line
+	3450 2725 3750 2725
+$Comp
+L power:GND #PWR03
+U 1 1 5E167AD3
+P 3750 3300
+AR Path="/5E167AD3" Ref="#PWR03"  Part="1"
+AR Path="/5E353BDD/5E167AD3" Ref="#PWR?"  Part="1"
+F 0 "#PWR03" H 3750 3050 50  0001 C CNN
+F 1 "GND" V 3755 3127 50  0000 C CNN
+F 2 "" H 3750 3300 50  0001 C CNN
+F 3 "" H 3750 3300 50  0001 C CNN
+	1    3750 3300
+	0    -1   1    0
+$EndComp
+Wire Wire Line
+	3450 3300 3750 3300
+$Comp
+L power:GND #PWR05
+U 1 1 5E169C3D
+P 3750 4800
+AR Path="/5E169C3D" Ref="#PWR05"  Part="1"
+AR Path="/5E353BDD/5E169C3D" Ref="#PWR?"  Part="1"
+F 0 "#PWR05" H 3750 4550 50  0001 C CNN
+F 1 "GND" V 3755 4627 50  0000 C CNN
+F 2 "" H 3750 4800 50  0001 C CNN
+F 3 "" H 3750 4800 50  0001 C CNN
+	1    3750 4800
+	0    -1   1    0
+$EndComp
+Wire Wire Line
+	3450 4800 3750 4800
+$Comp
+L power:+5V #PWR04
+U 1 1 5E16B5A5
+P 3750 3400
+F 0 "#PWR04" H 3750 3250 50  0001 C CNN
+F 1 "+5V" V 3765 3528 50  0000 L CNN
+F 2 "" H 3750 3400 50  0001 C CNN
+F 3 "" H 3750 3400 50  0001 C CNN
+	1    3750 3400
+	0    1    1    0
+$EndComp
+Wire Wire Line
+	3450 3400 3750 3400
+Text Label 3450 1325 0    50   ~ 0
+OFFSET_A
+Text Label 3450 1425 0    50   ~ 0
+OUTPUT_A
+Text Label 3450 1525 0    50   ~ 0
+OFFSET_B
+Text Label 3450 1625 0    50   ~ 0
+OUTPUT_B
+Text Label 3450 1725 0    50   ~ 0
+OFFSET_C
+Text Label 3450 1825 0    50   ~ 0
+OUTPUT_C
+Text Label 3450 1925 0    50   ~ 0
+OFFSET_D
+Text Label 3450 2025 0    50   ~ 0
+OUTPUT_D
+Text Label 3450 2125 0    50   ~ 0
+OUTPUT_E
+Text Label 3450 2225 0    50   ~ 0
+OUTPUT_F
+Text Label 3450 2325 0    50   ~ 0
+EXT_CLOCK_D
+Text Label 3450 2425 0    50   ~ 0
+INT_CLOCK_D
+Text Label 3450 2525 0    50   ~ 0
+STEP_PULSE_D
+Text Label 3450 3500 0    50   ~ 0
+SEQ_DIR_D
+Text Label 3450 3600 0    50   ~ 0
+SEQ_ZERO_D
+Text Label 3450 3700 0    50   ~ 0
+SEQ_RESET_D
+Text Label 3450 3800 0    50   ~ 0
+EXT_RATE_A
+Text Label 3450 3900 0    50   ~ 0
+PULSELEN_A
+Text Label 3450 4000 0    50   ~ 0
+EXT_POS_A
+NoConn ~ 3450 2625
+NoConn ~ 3450 4100
+NoConn ~ 3450 4200
+NoConn ~ 3450 4300
+NoConn ~ 3450 4400
+NoConn ~ 3450 4500
+NoConn ~ 3450 4600
+NoConn ~ 3450 4700
+Wire Wire Line
+	8100 825  8100 925
+Wire Wire Line
+	8100 825  7650 825
+Wire Wire Line
+	8100 925  7650 925
+Text Label 7650 825  0    50   ~ 0
+OUTPUT_E
+Text Label 7650 925  0    50   ~ 0
+OUTPUT_F
 $EndSCHEMATC

Commit message: Almost done now with both pcbs
Parts:
- added H1, H2, H3, H4: M3, MountingHole:MountingHole_3.2mm_M3_Pad, symbol Mechanical:MountingHole_Pad
- added J8: RIGHT, Connector_PinSocket_2.54mm:PinSocket_1x04_P2.54mm_Vertical, symbol Connector_Generic:Conn_01x04
- J1: footprint Connector_PinHeader_2.54mm:PinHeader_1x16_P2.54mm_Vertical -> Connector_PinSocket_2.54mm:PinSocket_1x16_P2.54mm_Vertical
- J2: footprint Connector_PinHeader_2.54mm:PinHeader_1x16_P2.54mm_Vertical -> Connector_PinSocket_2.54mm:PinSocket_1x08_P2.54mm_Vertical; symbol Connector_Generic:Conn_01x16 -> Connector_Generic:Conn_01x08
Connections:
- net +5V: now also J2.7 (Pin_7); no longer J2.15 (Pin_15)
- net EXT_POS_A: now also J8.1 (Pin_1); no longer J2.11 (Pin_11), J2.9 (Pin_9)
- net GND: now also J2.8 (Pin_8), H1.1, H2.1, H3.1, H4.1, J8.4 (Pin_4); no longer J2.16 (Pin_16)
- net OFFSET_A: no longer J1.14 (Pin_14)
- net OUTPUT_E: no longer J1.6 (Pin_6)
- net PULSELEN_A: now also J8.2 (Pin_2); no longer J2.10 (Pin_10)
- net SEQ_DIR_D: now also J2.6 (Pin_6); no longer J2.14 (Pin_14)
- net SEQ_RESET_D: now also J2.4 (Pin_4); no longer J2.12 (Pin_12)
- net SEQ_ZERO_D: now also J2.5 (Pin_5); no longer J2.13 (Pin_13)
- new net EXT_RATE_A: J8.3 (Pin_3)
- new net OUTPUT_A: J1.14 (Pin_14)
- new net OUTPUT_F: J1.6 (Pin_6)
- no-connect marks 8 -> 3
Changed lines of the file:
@@
 	9775 2150 10025 2150
-Wire Wire Line
-	8100 1950 8100 2050
 Wire Wire Line
 	8100 1950 7575 1950
@@
 $EndSheet
 Wire Wire Line
-	8950 825  8950 925
-Wire Wire Line
 	8950 825  9525 825
 Wire Wire Line
@@
 F 0 "J1" H 3168 1000 50  0000 C CNN
 F 1 "TOP" H 3168 1091 50  0000 C CNN
-F 2 "Connector_PinHeader_2.54mm:PinHeader_1x16_P2.54mm_Vertical" H 3250 2025 50  0001 C CNN
+F 2 "Connector_PinSocket_2.54mm:PinSocket_1x16_P2.54mm_Vertical" H 3250 2025 50  0001 C CNN
 F 3 "~" H 3250 2025 50  0001 C CNN
 	1    3250 2025
@@
 $EndComp
 $Comp
-L Connector_Generic:Conn_01x16 J2
+L Connector_Generic:Conn_01x08 J2
 U 1 1 5E162F36
-P 3250 4100
-F 0 "J2" H 3168 3075 50  0000 C CNN
-F 1 "BOTTOM" H 3168 3166 50  0000 C CNN
-F 2 "Connector_PinHeader_2.54mm:PinHeader_1x16_P2.54mm_Vertical" H 3250 4100 50  0001 C CNN
-F 3 "~" H 3250 4100 50  0001 C CNN
-	1    3250 4100
+P 3250 3700
+F 0 "J2" H 3175 3075 50  0000 C CNN
+F 1 "BOTTOM" H 3175 3175 50  0000 C CNN
+F 2 "Connector_PinSocket_2.54mm:PinSocket_1x08_P2.54mm_Vertical" H 3250 3700 50  0001 C CNN
+F 3 "~" H 3250 3700 50  0001 C CNN
+	1    3250 3700
 	-1   0    0    1
 $EndComp
@@
 L power:GND #PWR05
 U 1 1 5E169C3D
-P 3750 4800
+P 3750 4000
 AR Path="/5E169C3D" Ref="#PWR05"  Part="1"
 AR Path="/5E353BDD/5E169C3D" Ref="#PWR?"  Part="1"
-F 0 "#PWR05" H 3750 4550 50  0001 C CNN
-F 1 "GND" V 3755 4627 50  0000 C CNN
-F 2 "" H 3750 4800 50  0001 C CNN
-F 3 "" H 3750 4800 50  0001 C CNN
-	1    3750 4800
-	0    -1   1    0
-$EndComp
-Wire Wire Line
-	3450 4800 3750 4800
+F 0 "#PWR05" H 3750 3750 50  0001 C CNN
+F 1 "GND" V 3755 3827 50  0000 C CNN
+F 2 "" H 3750 4000 50  0001 C CNN
+F 3 "" H 3750 4000 50  0001 C CNN
+	1    3750 4000
+	0    -1   1    0
+$EndComp
+Wire Wire Line
+	3450 4000 3750 4000
 $Comp
 L power:+5V #PWR04
@@
 Text Label 3450 3700 0    50   ~ 0
 SEQ_RESET_D
-Text Label 3450 3800 0    50   ~ 0
+Text Label 3450 4675 0    50   ~ 0
 EXT_RATE_A
-Text Label 3450 3900 0    50   ~ 0
+Text Label 3450 4775 0    50   ~ 0
 PULSELEN_A
-Text Label 3450 4000 0    50   ~ 0
+Text Label 3450 4875 0    50   ~ 0
 EXT_POS_A
 NoConn ~ 3450 2625
-NoConn ~ 3450 4100
-NoConn ~ 3450 4200
-NoConn ~ 3450 4300
-NoConn ~ 3450 4400
-NoConn ~ 3450 4500
-NoConn ~ 3450 4600
-NoConn ~ 3450 4700
-Wire Wire Line
-	8100 825  8100 925
+NoConn ~ 3450 3800
+NoConn ~ 3450 3900
 Wire Wire Line
 	8100 825  7650 825
@@
 Text Label 7650 925  0    50   ~ 0
 OUTPUT_F
+$Comp
+L Mechanical:MountingHole_Pad H1
+U 1 1 5E195353
+P 1225 6625
+F 0 "H1" H 1325 6674 50  0000 L CNN
+F 1 "M3" H 1325 6583 50  0000 L CNN
+F 2 "MountingHole:MountingHole_3.2mm_M3_Pad" H 1225 6625 50  0001 C CNN
+F 3 "~" H 1225 6625 50  0001 C CNN
+	1    1225 6625
+	1    0    0    -1
+$EndComp
+$Comp
+L Mechanical:MountingHole_Pad H2
+U 1 1 5E195690
+P 1575 6625
+F 0 "H2" H 1675 6674 50  0000 L CNN
+F 1 "M3" H 1675 6583 50  0000 L CNN
+F 2 "MountingHole:MountingHole_3.2mm_M3_Pad" H 1575 6625 50  0001 C CNN
+F 3 "~" H 1575 6625 50  0001 C CNN
+	1    1575 6625
+	1    0    0    -1
+$EndComp
+$Comp
+L Mechanical:MountingHole_Pad H3
+U 1 1 5E195A0D
+P 1900 6625
+F 0 "H3" H 2000 6674 50  0000 L CNN
+F 1 "M3" H 2000 6583 50  0000 L CNN
+F 2 "MountingHole:MountingHole_3.2mm_M3_Pad" H 1900 6625 50  0001 C CNN
+F 3 "~" H 1900 6625 50  0001 C CNN
+	1    1900 6625
+	1    0    0    -1
+$EndComp
+$Comp
+L Mechanical:MountingHole_Pad H4
+U 1 1 5E195C5B
+P 2225 6625
+F 0 "H4" H 2325 6674 50  0000 L CNN
+F 1 "M3" H 2325 6583 50  0000 L CNN
+F 2 "MountingHole:MountingHole_3.2mm_M3_Pad" H 2225 6625 50  0001 C CNN
+F 3 "~" H 2225 6625 50  0001 C CNN
+	1    2225 6625
+	1    0    0    -1
+$EndComp
+$Comp
+L power:GND #PWR059
+U 1 1 5E195FDF
+P 1225 6725
+AR Path="/5E195FDF" Ref="#PWR059"  Part="1"
+AR Path="/5E353BDD/5E195FDF" Ref="#PWR?"  Part="1"
+F 0 "#PWR059" H 1225 6475 50  0001 C CNN
+F 1 "GND" V 1230 6552 50  0000 C CNN
+F 2 "" H 1225 6725 50  0001 C CNN
+F 3 "" H 1225 6725 50  0001 C CNN
+	1    1225 6725
+	-1   0    0    -1
+$EndComp
+$Comp
+L power:GND #PWR060
+U 1 1 5E19680B
+P 1575 6725
+AR Path="/5E19680B" Ref="#PWR060"  Part="1"
+AR Path="/5E353BDD/5E19680B" Ref="#PWR?"  Part="1"
+F 0 "#PWR060" H 1575 6475 50  0001 C CNN
+F 1 "GND" V 1580 6552 50  0000 C CNN
+F 2 "" H 1575 6725 50  0001 C CNN
+F 3 "" H 1575 6725 50  0001 C CNN
+	1    1575 6725
+	-1   0    0    -1
+$EndComp
+$Comp
+L power:GND #PWR061
+U 1 1 5E19694A
+P 1900 6725
+AR Path="/5E19694A" Ref="#PWR061"  Part="1"
+AR Path="/5E353BDD/5E19694A" Ref="#PWR?"  Part="1"
+F 0 "#PWR061" H 1900 6475 50  0001 C CNN
+F 1 "GND" V 1905 6552 50  0000 C CNN
+F 2 "" H 1900 6725 50  0001 C CNN
+F 3 "" H 1900 6725 50  0001 C CNN
+	1    1900 6725
+	-1   0    0    -1
+$EndComp
+$Comp
+L power:GND #PWR062
+U 1 1 5E196AD0
+P 2225 6725
+AR Path="/5E196AD0" Ref="#PWR062"  Part="1"
+AR Path="/5E353BDD/5E196AD0" Ref="#PWR?"  Part="1"
+F 0 "#PWR062" H 2225 6475 50  0001 C CNN
+F 1 "GND" V 2230 6552 50  0000 C CNN
+F 2 "" H 2225 6725 50  0001 C CNN
+F 3 "" H 2225 6725 50  0001 C CNN
+	1    2225 6725
+	-1   0    0    -1
+$EndComp
+$Comp
+L Connector_Generic:Conn_01x04 J8
+U 1 1 5E340773
+P 3250 4775
+F 0 "J8" H 3168 4350 50  0000 C CNN
+F 1 "RIGHT" H 3168 4441 50  0000 C CNN
+F 2 "Connector_PinSocket_2.54mm:PinSocket_1x04_P2.54mm_Vertical" H 3250 4775 50  0001 C CNN
+F 3 "~" H 3250 4775 50  0001 C CNN
+	1    3250 4775
+	-1   0    0    1
+$EndComp
+$Comp
+L power:GND #PWR067
+U 1 1 5E34FAC4
+P 3750 4575
+AR Path="/5E34FAC4" Ref="#PWR067"  Part="1"
+AR Path="/5E353BDD/5E34FAC4" Ref="#PWR?"  Part="1"
+F 0 "#PWR067" H 3750 4325 50  0001 C CNN
+F 1 "GND" V 3755 4402 50  0000 C CNN
+F 2 "" H 3750 4575 50  0001 C CNN
+F 3 "" H 3750 4575 50  0001 C CNN
+	1    3750 4575
+	0    -1   1    0
+$EndComp
+Wire Wire Line
+	3450 4575 3750 4575
 $EndSCHEMATC
