File: megasequencer/brain/brain/output_offset.sch (KiCad schematic (older format))
At the start: 30 parts, among them U7 TL074, U8 TL074

Commit message: Brain seem ok now, also start charting the program
Parts:
- added J7: FROM_OUTPUTS, Connector_PinHeader_2.54mm:PinHeader_1x06_P2.54mm_Vertical, symbol Connector_Generic:Conn_01x06
- renumbered C12 to C10, C13 to C11, C10 to C12, C11 to C13, R2 to R16, R3 to R17, R10 to R18, R11 to R19, R4 to R20, R12 to R21, R5 to R22, R13 to R23, R6 to R24, R14 to R25, R7 to R26, R15 to R27, R8 to R28, R9 to R29, R16 to R30, R17 to R31, R18 to R32, R19 to R33, R28 to R34, R29 to R35, R30 to R36, R31 to R37, R32 to R38, R33 to R39, U8 to U7, U7 to U8
Connections:
- net A_IN: no longer names the net of R32.2
- net A_IN: now also J7.1 (Pin_1)
- net B_IN: no longer names the net of R34.2
- net B_IN: now also J7.2 (Pin_2)
- net C_IN: no longer names the net of R36.2
- net C_IN: now also J7.3 (Pin_3)
- net D_IN: no longer names the net of R38.2
- net D_IN: now also J7.4 (Pin_4)
- new net E_OUT: J7.5 (Pin_5)
- new net F_OUT: J7.6 (Pin_6)
