File: offsetscaler/offsetscaler-panel/offsetscaler-panel.kicad_pcb (KiCad board)
At the start: 2 copper layers, 66 x 99.1 mm, 6 parts

Commit message: All holes done
Parts:
- added REF**: MountingHole_5mm, MountingHole:MountingHole_5mm, F.Cu at (153.7, 105.9)
- added REF**: MountingHole_6mm, MountingHole:MountingHole_6mm, F.Cu at (150.0, 152.9)
- added REF**: MountingHole_5mm, MountingHole:MountingHole_5mm, F.Cu at (144.8, 105.9)
- added REF**: MountingHole_5mm, MountingHole:MountingHole_5mm, F.Cu at (153.7, 119.9)
- added REF**: MountingHole_5mm, MountingHole:MountingHole_5mm, F.Cu at (144.8, 119.9)
- added REF**: MountingHole_6mm, MountingHole:MountingHole_6mm, F.Cu at (150.0, 72.9)
- added REF**: MountingHole_6mm, MountingHole:MountingHole_6mm, F.Cu at (150.0, 84.3)
- added REF**: MountingHole_6mm, MountingHole:MountingHole_6mm, F.Cu at (150.0, 95.8)
- added REF**: MountingHole_6mm, MountingHole:MountingHole_6mm, F.Cu at (150.0, 130.0)
- added REF**: MountingHole_6mm, MountingHole:MountingHole_6mm, F.Cu at (150.0, 141.5)
Other:
- board text added: "k"
- board text added: "m"
- board text added: "x"
- board text added: "y"
- board text added: "y = k(x + m)"
- board text added: "~y"
Changed lines of the file:
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@@
   (general
     (thickness 1.6)
-    (drawings 4)
+    (drawings 15)
     (tracks 0)
     (zones 0)
-    (modules 6)
+    (modules 16)
     (nets 1)
   )
@@
     (uvia_drill 0.1)
   )
+  (module MountingHole:MountingHole_5mm (layer F.Cu)
+    (at 153.67 105.918)
+    (descr "Mounting Hole 5mm, no annular")
+    (tags "mounting hole 5mm no annular")
+    (attr virtual)
+    (fp_text reference REF** (at 0 -6) (layer F.SilkS) hide
+      (effects (font (size 1 1) (thickness 0.15)))
+    )
+    (fp_text value MountingHole_5mm (at 0 6) (layer F.Fab) hide
+      (effects (font (size 1 1) (thickness 0.15)))
+    )
+    (fp_text user %R (at 0.3 0) (layer F.Fab) hide
+      (effects (font (size 1 1) (thickness 0.15)))
+    )
+    (fp_circle (center 0 0) (end 5 0) (layer Cmts.User) (width 0.15))
+    (fp_circle (center 0 0) (end 5.25 0) (layer F.CrtYd) (width 0.05))
+    (pad 1 np_thru_hole circle (at 0 0) (size 5 5) (drill 5) (layers *.Cu *.Mask))
+  )
+  (module MountingHole:MountingHole_5mm (layer F.Cu)
+    (at 144.78 105.918)
+    (descr "Mounting Hole 5mm, no annular")
+    (tags "mounting hole 5mm no annular")
+    (attr virtual)
+    (fp_text reference REF** (at 0 -6) (layer F.SilkS) hide
+      (effects (font (size 1 1) (thickness 0.15)))
+    )
+    (fp_text value MountingHole_5mm (at 0 6) (layer F.Fab) hide
+      (effects (font (size 1 1) (thickness 0.15)))
+    )
+    (fp_circle (center 0 0) (end 5.25 0) (layer F.CrtYd) (width 0.05))
+    (fp_circle (center 0 0) (end 5 0) (layer Cmts.User) (width 0.15))
+    (fp_text user %R (at 0.3 0) (layer F.Fab) hide
+      (effects (font (size 1 1) (thickness 0.15)))
+    )
+    (pad 1 np_thru_hole circle (at 0 0) (size 5 5) (drill 5) (layers *.Cu *.Mask))
+  )
+  (module MountingHole:MountingHole_5mm (layer F.Cu)
+    (at 153.67 119.888)
+    (descr "Mounting Hole 5mm, no annular")
+    (tags "mounting hole 5mm no annular")
+    (attr virtual)
+    (fp_text reference REF** (at 0 -6) (layer F.SilkS) hide
+      (effects (font (size 1 1) (thickness 0.15)))
+    )
+    (fp_text value MountingHole_5mm (at 0 6) (layer F.Fab) hide
+      (effects (font (size 1 1) (thickness 0.15)))
+    )
+    (fp_text user %R (at 0.3 0) (layer F.Fab) hide
+      (effects (font (size 1 1) (thickness 0.15)))
+    )
+    (fp_circle (center 0 0) (end 5 0) (layer Cmts.User) (width 0.15))
+    (fp_circle (center 0 0) (end 5.25 0) (layer F.CrtYd) (width 0.05))
+    (pad 1 np_thru_hole circle (at 0 0) (size 5 5) (drill 5) (layers *.Cu *.Mask))
+  )
+  (module MountingHole:MountingHole_5mm (layer F.Cu)
+    (at 144.78 119.888)
+    (descr "Mounting Hole 5mm, no annular")
+    (tags "mounting hole 5mm no annular")
+    (attr virtual)
+    (fp_text reference REF** (at 0 -6) (layer F.SilkS) hide
+      (effects (font (size 1 1) (thickness 0.15)))
+    )
+    (fp_text value MountingHole_5mm (at 0 6) (layer F.Fab) hide
+      (effects (font (size 1 1) (thickness 0.15)))
+    )
+    (fp_circle (center 0 0) (end 5.25 0) (layer F.CrtYd) (width 0.05))
+    (fp_circle (center 0 0) (end 5 0) (layer Cmts.User) (width 0.15))
+    (fp_text user %R (at 0.3 0) (layer F.Fab) hide
+      (effects (font (size 1 1) (thickness 0.15)))
+    )
+    (pad 1 np_thru_hole circle (at 0 0) (size 5 5) (drill 5) (layers *.Cu *.Mask))
+  )
+  (module MountingHole:MountingHole_6mm (layer F.Cu)
+    (at 149.98954 72.898)
+    (descr "Mounting Hole 6mm, no annular")
+    (tags "mounting hole 6mm no annular")
+    (attr virtual)
+    (fp_text reference REF** (at 0 -7) (layer F.SilkS) hide
+      (effects (font (size 1 1) (thickness 0.15)))
+    )
+    (fp_text value MountingHole_6mm (at 0 7) (layer F.Fab) hide
+      (effects (font (size 1 1) (thickness 0.15)))
+    )
+    (fp_circle (center 0 0) (end 6.25 0) (layer F.CrtYd) (width 0.05))
+    (fp_circle (center 0 0) (end 6 0) (layer Cmts.User) (width 0.15))
+    (fp_text user %R (at 0.3 0) (layer F.Fab) hide
+      (effects (font (size 1 1) (thickness 0.15)))
+    )
+    (pad 1 np_thru_hole circle (at 0 0) (size 6 6) (drill 6) (layers *.Cu *.Mask))
+  )
+  (module MountingHole:MountingHole_6mm (layer F.Cu)
+    (at 149.98954 84.328)
+    (descr "Mounting Hole 6mm, no annular")
+    (tags "mounting hole 6mm no annular")
+    (attr virtual)
+    (fp_text reference REF** (at 0 -7) (layer F.SilkS) hide
+      (effects (font (size 1 1) (thickness 0.15)))
+    )
+    (fp_text value MountingHole_6mm (at 0 7) (layer F.Fab) hide
+      (effects (font (size 1 1) (thickness 0.15)))
+    )
+    (fp_text user %R (at 0.3 0) (layer F.Fab) hide
+      (effects (font (size 1 1) (thickness 0.15)))
+    )
+    (fp_circle (center 0 0) (end 6 0) (layer Cmts.User) (width 0.15))
+    (fp_circle (center 0 0) (end 6.25 0) (layer F.CrtYd) (width 0.05))
+    (pad 1 np_thru_hole circle (at 0 0) (size 6 6) (drill 6) (layers *.Cu *.Mask))
+  )
+  (module MountingHole:MountingHole_6mm (layer F.Cu)
+    (at 149.98954 95.758)
+    (descr "Mounting Hole 6mm, no annular")
+    (tags "mounting hole 6mm no annular")
+    (attr virtual)
+    (fp_text reference REF** (at 0 -7) (layer F.SilkS) hide
+      (effects (font (size 1 1) (thickness 0.15)))
+    )
+    (fp_text value MountingHole_6mm (at 0 7) (layer F.Fab) hide
+      (effects (font (size 1 1) (thickness 0.15)))
+    )
+    (fp_circle (center 0 0) (end 6.25 0) (layer F.CrtYd) (width 0.05))
+    (fp_circle (center 0 0) (end 6 0) (layer Cmts.User) (width 0.15))
+    (fp_text user %R (at 0.3 0) (layer F.Fab) hide
+      (effects (font (size 1 1) (thickness 0.15)))
+    )
+    (pad 1 np_thru_hole circle (at 0 0) (size 6 6) (drill 6) (layers *.Cu *.Mask))
+  )
+  (module MountingHole:MountingHole_6mm (layer F.Cu)
+    (at 149.98954 130.048)
+    (descr "Mounting Hole 6mm, no annular")
+    (tags "mounting hole 6mm no annular")
+    (attr virtual)
+    (fp_text reference REF** (at 0 -7) (layer F.SilkS) hide
+      (effects (font (size 1 1) (thickness 0.15)))
+    )
+    (fp_text value MountingHole_6mm (at 0 7) (layer F.Fab) hide
+      (effects (font (size 1 1) (thickness 0.15)))
+    )
+    (fp_text user %R (at 0.3 0) (layer F.Fab) hide
+      (effects (font (size 1 1) (thickness 0.15)))
+    )
+    (fp_circle (center 0 0) (end 6 0) (layer Cmts.User) (width 0.15))
+    (fp_circle (center 0 0) (end 6.25 0) (layer F.CrtYd) (width 0.05))
+    (pad 1 np_thru_hole circle (at 0 0) (size 6 6) (drill 6) (layers *.Cu *.Mask))
+  )
+  (module MountingHole:MountingHole_6mm (layer F.Cu)
+    (at 149.98954 141.478)
+    (descr "Mounting Hole 6mm, no annular")
+    (tags "mounting hole 6mm no annular")
+    (attr virtual)
+    (fp_text reference REF** (at 0 -7) (layer F.SilkS) hide
+      (effects (font (size 1 1) (thickness 0.15)))
+    )
+    (fp_text value MountingHole_6mm (at 0 7) (layer F.Fab) hide
+      (effects (font (size 1 1) (thickness 0.15)))
+    )
+    (fp_circle (center 0 0) (end 6.25 0) (layer F.CrtYd) (width 0.05))
+    (fp_circle (center 0 0) (end 6 0) (layer Cmts.User) (width 0.15))
+    (fp_text user %R (at 0.3 0) (layer F.Fab) hide
+      (effects (font (size 1 1) (thickness 0.15)))
+    )
+    (pad 1 np_thru_hole circle (at 0 0) (size 6 6) (drill 6) (layers *.Cu *.Mask))
+  )
+  (module MountingHole:MountingHole_6mm (layer F.Cu)
+    (at 149.98954 152.908)
+    (descr "Mounting Hole 6mm, no annular")
+    (tags "mounting hole 6mm no annular")
+    (attr virtual)
+    (fp_text reference REF** (at 0 -7) (layer F.SilkS) hide
+      (effects (font (size 1 1) (thickness 0.15)))
+    )
+    (fp_text value MountingHole_6mm (at 0 7) (layer F.Fab) hide
+      (effects (font (size 1 1) (thickness 0.15)))
+    )
+    (fp_circle (center 0 0) (end 6.25 0) (layer F.CrtYd) (width 0.05))
+    (fp_circle (center 0 0) (end 6 0) (layer Cmts.User) (width 0.15))
+    (fp_text user %R (at 0.3 0) (layer F.Fab) hide
+      (effects (font (size 1 1) (thickness 0.15)))
+    )
+    (pad 1 np_thru_hole circle (at 0 0) (size 6 6) (drill 6) (layers *.Cu *.Mask))
+  )
   (module 3296W-1-250:MountingHole_Pot_Alp (layer F.Cu)
     (at 182.92064 77.84338)
@@
     (pad 1 np_thru_hole circle (at 0 0) (size 3.2 3.2) (drill 3.2) (layers *.Cu *.Mask))
   )
+  (gr_text "y = k(x + m)" (at 166.878 113.03) (layer F.SilkS)
+    (effects (font (size 3.048 3.048) (thickness 0.762) italic) (justify left))
+  )
+  (gr_text m (at 169.164 77.47) (layer F.SilkS)
+    (effects (font (size 3.048 3.048) (thickness 0.5842)) (justify left))
+  )
+  (gr_text m (at 169.164 127.762) (layer F.SilkS)
+    (effects (font (size 3.048 3.048) (thickness 0.5842)) (justify left))
+  )
+  (gr_text k (at 169.164 147.32) (layer F.SilkS)
+    (effects (font (size 3.048 3.048) (thickness 0.5842)) (justify left))
+  )
+  (gr_text k (at 168.91 97.536) (layer F.SilkS)
+    (effects (font (size 3.048 3.048) (thickness 0.5842)) (justify left))
+  )
+  (gr_text y (at 157.48 152.654) (layer F.SilkS)
+    (effects (font (size 3.048 3.048) (thickness 0.5842)) (justify left))
+  )
+  (gr_text ~y (at 157.48 141.224) (layer F.SilkS)
+    (effects (font (size 3.048 3.048) (thickness 0.5842)) (justify left))
+  )
+  (gr_text x (at 157.48 129.794) (layer F.SilkS)
+    (effects (font (size 3.048 3.048) (thickness 0.5842)) (justify left))
+  )
+  (gr_text y (at 157.48 95.504) (layer F.SilkS)
+    (effects (font (size 3.048 3.048) (thickness 0.5842)) (justify left))
+  )
+  (gr_text ~y (at 157.48 84.074) (layer F.SilkS)
+    (effects (font (size 3.048 3.048) (thickness 0.5842)) (justify left))
+  )
+  (gr_text x (at 157.48 72.644) (layer F.SilkS)
+    (effects (font (size 3.048 3.048) (thickness 0.5842)) (justify left))
+  )
   (gr_line (start 139.7 162.56) (end 139.7 63.5) (layer Edge.Cuts) (width 0.05))
