File: roaster/roaster.sch (KiCad schematic (older format))
At the start: 26 parts, among them J1 PWR_IN, J2 SPI, J3 DISP, J4 UART, J5 THERM, J6 FAN, J7 HEAT, SW1 SW_RST, SW2 SW_STOP_MODE, SW3 SW_START_SET, U1 ATmega328P-PU, Y1 16MHz

Commit message: Add print panel graphics
Parts:
- U1: symbol MCU_Microchip_ATmega:ATmega328P-PU -> roaster-rescue:ATmega328P-PU-MCU_Microchip_ATmega
Changed lines of the file:
@@
 $EndDescr
 $Comp
-L MCU_Microchip_ATmega:ATmega328P-PU U1
+L roaster-rescue:ATmega328P-PU-MCU_Microchip_ATmega U1
 U 1 1 5E9CAAAF
 P 2400 3350
