File: megasequencer/interface/interface.kicad_pcb (KiCad board)
At the start: 2 copper layers, 99.1 x 99.1 mm, 56 parts, among them J1 INT_CLOCK_OUT, J10 OFFSET_A, J11 OFFSET_B, J12 OFFSET_C, J13 OFFSET_D, J14 OUTPUT_A, J15 OUTPUT_B, J16 OUTPUT_C, J17 OUTPUT_D, J18 OUTPUT_E, J19 OUTPUT_F, J2 EXT_CLOCK_IN, J20 TOP, J21 BOTTOM, J22 RIGHT, J3 DIR_IN, J4 RESET_IN, J5 ZERO_IN, J6 STEP_OUT, J7 EXT_RATE_CV, J8 EXT_POS_CV, J9 PULSELEN_CV, SW1 CLOCK_SW, SW2 RESET_SW, SW3 ZERO_SW, SW4 SEQ_DIR

Commit message: Wrong LED direction
Parts:
- moved D1 2.54 mm to (104.1, 31.8), turned to 180 degrees
- moved D2 2.54 mm to (115.6, 31.8), turned to 180 degrees
Connections:
- D1 pad 1: /INT_CLOCK_D -> GND
- D1 pad 2: GND -> /INT_CLOCK_D
- D2 pad 1: /STEP_PULSE_D -> GND
- D2 pad 2: GND -> /STEP_PULSE_D
