File: vca/vca/vca.kicad_pcb (KiCad board)
At the start: 2 copper layers, 99.1 x 99.1 mm, 106 parts, among them J1 CV1, J10 OUT1, J11 OUT2, J12 OUT3, J13 OUT4, J14 OUTMIX, J2 CV2, J3 CV3, J4 CV4, J5 POWER, J6 IN4, J7 IN3, J8 IN2, J9 IN1, U1 TL084, U2 SSI2164, U3 TL084, U4 TL072

Commit message: Route the VCA
Parts:
- C1, C2, J5: moved to B.Cu
- moved J5 3.81 mm to (132.1, 123.2), turned to 180 degrees
- renumbered C15 to Cr, R34 to Rw
Routing:
- net -12V: track 0.00 -> 226.0 mm
- net +12V: track 0.00 -> 173.5 mm
- net Net-(C15-Pad2): track 0.00 -> 113.1 mm
- net Net-(R15-Pad1): track 0.00 -> 91.7 mm
- net Net-(J10-PadT): track 0.00 -> 86.3 mm
- net Net-(J8-PadT): track 0.00 -> 85.1 mm
- net Net-(C16-Pad2): track 0.00 -> 84.2 mm
- net Net-(C19-Pad2): track 0.00 -> 82.8 mm
- net Net-(R10-Pad1): track 0.00 -> 80.1 mm
- net Net-(J9-PadT): track 0.00 -> 73.8 mm
- net Net-(R12-Pad1): track 0.00 -> 73.3 mm
- net Net-(J7-PadT): track 0.00 -> 65.7 mm
- net Net-(J11-PadT): track 0.00 -> 65.6 mm
- net Net-(R13-Pad1): track 0.00 -> 64.0 mm
- net Net-(C18-Pad2): track 0.00 -> 54.3 mm
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- added copper zone on B.Cu, net GND
- added copper zone on F.Cu, net GND
Other:
- board text added: "2021-04-18"
- board text added: "QUAD VCA W/ MIXER"
- board text added: "RED LINE -12V"
