File: lfo/lfo.sch (KiCad schematic (older format))
At the start: 70 parts, among them J1 CV, J2 Conn_02x05_Odd_Even, J3 TRI, J4 SQR, J5 RAMP UP, J6 SIN, J7 COS, J8 RAMP DOWN, Q1 BC550, Q2 BC550, Q3 BC550, Q4 BC550, Q5 BC550, U1 TL074, U2 TL074, U3 TL072

Commit message: Fix bugs and add footprints
Parts:
- added D2, D3: 1N4004, Diode_THT:D_5W_P12.70mm_Horizontal, symbol Device:D
- added R41: 100k, Resistor_THT:R_Axial_DIN0204_L3.6mm_D1.6mm_P7.62mm_Horizontal, symbol Device:R
- added R42, R43: 10R, Resistor_THT:R_Axial_DIN0204_L3.6mm_D1.6mm_P7.62mm_Horizontal, symbol Device:R
- added R44: 10K, Resistor_THT:R_Axial_DIN0204_L3.6mm_D1.6mm_P7.62mm_Horizontal, symbol Device:R
- C1, C2, C3, C4, C5, C6, C7: footprint (none) -> Capacitor_THT:C_Disc_D5.0mm_W2.5mm_P2.50mm
- C8, C9: footprint (none) -> Capacitor_THT:CP_Radial_D5.0mm_P2.00mm
- D1: footprint (none) -> LED_THT:LED_D3.0mm
- J1, J3, J4, J5, J6, J7, J8: footprint (none) -> Connector_Audio:Jack_3.5mm_QingPu_WQP-PJ398SM_Vertical_CircularHoles
- J2: value Conn_02x05_Odd_Even -> EURO; footprint (none) -> Connector_PinHeader_2.54mm:PinHeader_2x05_P2.54mm_Vertical
- R1, R10, R11, R12, R13, R14, R15, R16, R17, R18, R19, R2, R20, R21, R22, R23, R25, R26, R27, R28, R29, R3, R30, R31, R32, R34, R35, R36, R37, R38, R39, R4, R40, R5, R6, R7, R8, R9: footprint (none) -> Resistor_THT:R_Axial_DIN0204_L3.6mm_D1.6mm_P7.62mm_Horizontal
- R24: value 58K -> 68K; footprint (none) -> Resistor_THT:R_Axial_DIN0204_L3.6mm_D1.6mm_P7.62mm_Horizontal
- R33: value 20K -> RAMP 20K; footprint (none) -> Resistor_THT:R_Axial_DIN0204_L3.6mm_D1.6mm_P7.62mm_Horizontal
- RV1, RV2: footprint (none) -> Potentiometer_THT:Potentiometer_Alps_RK09L_Single_Vertical
- RV3: value CV -> SC1 100K; footprint (none) -> Potentiometer_THT:Potentiometer_Bourns_3296W_Vertical
- RV4: value CV -> SC2 50K; footprint (none) -> Potentiometer_THT:Potentiometer_Bourns_3296W_Vertical
- U1, U2: footprint (none) -> Package_DIP:DIP-14_W7.62mm_Socket_LongPads
- U3: footprint (none) -> Package_DIP:DIP-8_W7.62mm_Socket_LongPads
Connections:
- net +12V: now also D2.1 (K), R42.2; no longer C8.1, J2.1 (Pin_1), J2.2 (Pin_2)
- net -12V: now also D3.2 (A), R43.2; no longer C9.2, J2.10 (Pin_10), J2.9 (Pin_9)
- net GND: now also Q1.3 (E), Q4.3 (E), D2.2 (A), D3.1 (K); no longer Q1.1 (C), Q4.1 (C)
- net at R3.2, U1.1: now also R41.1
- net at R1.1, R2.1, U1.2 (-): now also R41.2
- net at R22.1, U2.3 (+): now also Q4.1 (C); no longer Q4.3 (E)
- net at R19.1, R29.1, U3.2 (-): now also Q3.1 (C); no longer Q3.3 (E)
- net at R25.1, R28.2, U3.3 (+): now also Q5.1 (C); no longer Q5.3 (E)
- net at R32.1, U3.6 (-): now also R44.2
- net at R39.1, U3.7: now also R44.1
- net at R23.2, RV4.3: now also Q3.3 (E); no longer Q3.1 (C)
- net at R23.1, RV4.1: now also Q5.3 (E); no longer Q5.1 (C)
- net at R7.1: now also Q1.1 (C); no longer Q1.3 (E)
- net at Q2.1 (C): now also D1.1 (K); no longer R12.1
- net at Q2.3 (E): now also R12.1; no longer D1.1 (K)
- new net: C8.1, J2.1 (Pin_1), J2.2 (Pin_2), R42.1
- new net: C9.2, J2.10 (Pin_10), J2.9 (Pin_9), R43.1

Commit message: Start fiddling with the PCB for the VCLFO
Parts:
- R33: footprint Resistor_THT:R_Axial_DIN0204_L3.6mm_D1.6mm_P7.62mm_Horizontal -> Potentiometer_THT:Potentiometer_Bourns_3296W_Vertical
Changed lines of the file:
@@
 F 0 "R33" V 9050 5250 50  0000 C CNN
 F 1 "RAMP 20K" V 8950 5250 50  0000 C CNN
-F 2 "Resistor_THT:R_Axial_DIN0204_L3.6mm_D1.6mm_P7.62mm_Horizontal" V 8730 5250 50  0001 C CNN
+F 2 "Potentiometer_THT:Potentiometer_Bourns_3296W_Vertical" V 8730 5250 50  0001 C CNN
 F 3 "~" H 8800 5250 50  0001 C CNN
 	1    8800 5250
