File: lfo/lfo.kicad_pcb (KiCad board)
At the start: 2 copper layers, 76 parts, among them J1 CV, J2 EURO, J3 TRI, J4 SQR, J5 RAMP UP, J6 SIN, J7 COS, J8 RAMP DOWN, Q1 BC550, Q2 BC550, Q3 BC550, Q4 BC550, Q5 BC550, U1 TL074, U2 TL074, U3 TL072

Commit message: Place all the stuffs
Parts:
- C1, C2, C3, C4, C5, C6, C8, C9, D2, D3, J2, Q3, Q5, R15, R17, R19, R23, R24, R25, R27, R28, R29, R30, R31, R32, R35, R36, R38, R42, R43, R44: moved to B.Cu
- moved R38 207.9 mm to (68.6, 94.6)
- moved C4 203.4 mm to (73.0, 102.2)
- moved C2 202.4 mm to (73.0, 75.6)
- moved R36 189.5 mm to (76.2, 97.2), turned to 180 degrees
- moved C1 184.3 mm to (90.8, 76.2)
- moved R30 182.9 mm to (90.2, 108.0)
- moved R17 171.2 mm to (76.2, 105.4), turned to 180 degrees
- moved C3 168.5 mm to (90.8, 102.2)
- moved Q3 167.2 mm to (104.1, 118.7)
- moved C5 166.8 mm to (111.8, 98.4)
- moved R33 165.3 mm to (73.0, 118.7), turned to 180 degrees
- moved RV3 163.1 mm to (94.6, 118.7), turned to 180 degrees
- moved R19 155.1 mm to (101.0, 102.2)
- moved R32 153.5 mm to (108.6, 107.3), turned to 180 degrees
- moved R31 149.7 mm to (97.8, 105.4), turned to 180 degrees
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Other:
- board outline added: 99.1 x 99.1 mm
- board text added: "RED LINE -12V"

Commit message: Route the VCLFO
Parts:
- moved C8 34.3 mm to (142.2, 73.0)
- moved C9 32.4 mm to (142.1, 109.2)
- moved C6 2.54 mm to (125.7, 110.5), turned to 180 degrees
- moved R10 1.91 mm to (90.2, 88.9)
Routing:
- net -12V: track 0.00 -> 176.5 mm
- net +12V: track 0.00 -> 158.6 mm
- net Net-(C7-Pad1): track 0.00 -> 88.7 mm
- net Net-(R11-Pad1): track 0.00 -> 88.0 mm
- net Net-(Q3-Pad1): track 0.00 -> 64.2 mm
- net Net-(J1-PadT): track 0.00 -> 62.2 mm
- net Net-(R1-Pad2): track 0.00 -> 50.6 mm
- net Net-(R29-Pad2): track 0.00 -> 50.2 mm
- net Net-(R38-Pad2): track 0.00 -> 43.9 mm
- net Net-(R39-Pad1): track 0.00 -> 43.6 mm
- net Net-(R35-Pad2): track 0.00 -> 43.5 mm
- net Net-(Q4-Pad1): track 0.00 -> 31.4 mm
- net Net-(C9-Pad2): track 0.00 -> 30.5 mm
- net Net-(C8-Pad1): track 0.00 -> 29.4 mm
- net Net-(R13-Pad2): track 0.00 -> 29.1 mm
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- added copper zone on B.Cu, net GND
- added copper zone on F.Cu, net GND
Other:
- board text added: "VCLFO SKULL AND CIRCUIT 2021-10-05"

Commit message: Fix
Parts:
- added REF**: MountingHole_3.2mm_M3, MountingHole:MountingHole_3.2mm_M3, F.Cu at (151.1, 135.9)
- added REF**: MountingHole_3.2mm_M3, MountingHole:MountingHole_3.2mm_M3, F.Cu at (151.1, 73.0)
- added REF**: MountingHole_3.2mm_M3, MountingHole:MountingHole_3.2mm_M3, F.Cu at (130.8, 52.1)
