File: vcf/vcf/vcf.sch (KiCad schematic (older format))
At the start: 80 parts, among them J1 1V/Oct, J2 CVF, J3 CVR, J4 AUDIO IN, J5 EURO, J6 AUDIO OUT, SW1 SW_SPST ON-ON, U1 TL072, U2 TL072, U3 AS3320, U4 4066, U5 4066

Commit message: Time to route
Parts:
- J5: footprint Connector_Audio:Jack_3.5mm_QingPu_WQP-PJ398SM_Vertical_CircularHoles -> Connector_PinHeader_2.54mm:PinHeader_2x05_P2.54mm_Vertical
Changed lines of the file:
@@
 F 0 "J5" H 7900 10417 50  0000 C CNN
 F 1 "EURO" H 7900 10326 50  0000 C CNN
-F 2 "Connector_Audio:Jack_3.5mm_QingPu_WQP-PJ398SM_Vertical_CircularHoles" H 7850 10000 50  0001 C CNN
+F 2 "Connector_PinHeader_2.54mm:PinHeader_2x05_P2.54mm_Vertical" H 7850 10000 50  0001 C CNN
 F 3 "~" H 7850 10000 50  0001 C CNN
 	1    7850 10000
