File: vcf/vcf/vcf.kicad_pcb (KiCad board)
At the start: 2 copper layers, 99.1 x 99.1 mm, 80 parts, among them J1 1V/Oct, J2 CVF, J3 CVR, J4 AUDIO IN, J5 EURO, J6 AUDIO OUT, SW1 SW_SPST ON-ON, U1 TL072, U2 TL072, U3 AS3320, U4 4066, U5 4066

Commit message: Time to route
Parts:
- R1, R10, R11, R12, R13, R14, R15, R16, R17, R18, R19, R2, R20, R21, R22, R23, R24, R25, R26, R27, R28, R29, R3, R30, R31, R32, R33, R34, R36, R38, R39, R4, R40, R5, R6, R7, R8, R9: moved to B.Cu
- moved R3 210.1 mm to (55.9, 92.7)
- moved R29 207.8 mm to (55.9, 95.2)
- moved R12 196.7 mm to (72.4, 71.8), turned to 90 degrees
- moved R13 191.3 mm to (68.6, 64.1), turned to 270 degrees
- moved R4 190.8 mm to (56.5, 75.6), turned to 90 degrees
- moved R18 190.2 mm to (85.1, 88.9), turned to 90 degrees
- moved R38 190.2 mm to (77.5, 85.7), turned to 270 degrees
- moved R35 184.2 mm to (72.4, 88.3)
- moved R10 183.9 mm to (74.9, 71.8), turned to 90 degrees
- moved R17 183.7 mm to (82.5, 91.4), turned to 270 degrees
- moved R15 170.0 mm to (63.5, 97.8), turned to 180 degrees
- moved R28 168.5 mm to (99.7, 81.3)
- moved R1 168.4 mm to (43.8, 66.0)
- moved R21 168.2 mm to (82.5, 113.0), turned to 270 degrees
- moved R33 167.2 mm to (85.7, 78.1), turned to 90 degrees
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
Commit message: The VCF is routed. Finally
Parts:
- moved R28 69.5 mm to (55.9, 135.3)
- moved RV9 52.8 mm to (78.7, 127.6)
- moved R29 28.6 mm to (55.9, 123.8)
- moved C11 11.5 mm to (69.8, 135.3), turned to 90 degrees
- moved C12 8.98 mm to (69.8, 126.4), turned to 90 degrees
- moved D1 8.89 mm to (55.9, 132.7)
- moved D2 8.89 mm to (55.9, 126.4)
Routing:
- net +12V: track 0.00 -> 361.7 mm
- net -12V: track 0.00 -> 252.3 mm
- net Net-(R11-Pad2): track 0.00 -> 211.1 mm
- net Net-(R20-Pad2): track 0.00 -> 109.2 mm
- net Net-(R8-Pad2): track 0.00 -> 103.0 mm
- net Net-(C14-Pad2): track 0.00 -> 95.6 mm
- net Net-(R38-Pad1): track 0.00 -> 87.0 mm
- net Net-(D3-Pad1): track 0.00 -> 80.0 mm
- net Net-(C10-Pad2): track 0.00 -> 69.9 mm
- net Net-(R1-Pad2): track 0.00 -> 64.0 mm
- net Net-(R12-Pad2): track 0.00 -> 62.1 mm
- net Net-(R14-Pad2): track 0.00 -> 60.5 mm
- net Net-(J2-PadT): track 0.00 -> 59.1 mm
- net Net-(C14-Pad1): track 0.00 -> 55.9 mm
- net Net-(R16-Pad2): track 0.00 -> 55.7 mm
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