File: vcf/vcf/vcf.kicad_pcb (KiCad board)
At the start: 2 copper layers, 99.1 x 99.1 mm, 80 parts, among them J1 1V/Oct, J2 CVF, J3 CVR, J4 AUDIO IN, J5 EURO, J6 AUDIO OUT, SW1 SW_SPST ON-ON, U1 TL072, U2 TL072, U3 AS3320, U4 4066, U5 4066

Commit message: KiCad 6.0 upgrade
Other:
- net class Default removed
