File: noise/noise/noise.kicad_pcb (KiCad board)
At the start: 2 copper layers, 33 x 99.1 mm, 38 parts, among them J1 Out1, J2 Out2, J3 Out3, J4 Out4, J5 POWER, Q1 2N3904, Q2 2N3904, Q3 2N3904, Q4 2N3904, U1 TL074

Commit message: Add 8bit dvco and update some project files
Other:
- net class Default removed
