File: 8bitdvco/8bitdvco.kicad_sch (KiCad schematic)
At the start: 87 parts, among them J1 DO, J2 SPI, J3 PWR, J4 DI, J5 SLIDER12, J6 SLIDER34, J7 SLIDER50, J8 OUTPUTS, J9 BUTTONS, Q1 2N3904, SW1 SW_RST, U1 ATmega328P-PU, U2 L78L05_TO92, U3 TL074, U4 TL074, Y1 16MHz

Commit message: done without errors and warnings
Parts:
- C13, C14: footprint (none) -> Capacitor_THT:C_Disc_D3.0mm_W1.6mm_P2.50mm
- D4, D5: footprint (none) -> Diode_THT:D_DO-35_SOD27_P7.62mm_Horizontal
- FB1, FB2: footprint (none) -> Resistor_THT:R_Axial_DIN0309_L9.0mm_D3.2mm_P12.70mm_Horizontal
- J5, J6: footprint (none) -> Connector_PinHeader_2.54mm:PinHeader_1x02_P2.54mm_Vertical
- J7, J8: footprint (none) -> Connector_PinHeader_2.54mm:PinHeader_1x03_P2.54mm_Vertical
- J9: footprint (none) -> Connector_PinHeader_2.54mm:PinHeader_1x06_P2.54mm_Vertical
- R10, R11, R12, R13, R14, R15, R16, R17, R18, R19, R20, R21, R22, R23, R24, R25, R26, R27, R28, R29, R30, R31, R32, R33, R34, R35, R36, R37, R38, R39, R4, R5, R6, R7, R8, R9: footprint Resistor_THT:R_Axial_DIN0411_L9.9mm_D3.6mm_P12.70mm_Horizontal -> Resistor_THT:R_Axial_DIN0204_L3.6mm_D1.6mm_P7.62mm_Horizontal
- U4: footprint (none) -> Package_DIP:DIP-14_W7.62mm_LongPads
